Commit message: add point_cloud segmentation files

File: catkin_ws/src/site/urdf/deepracer.urdf (robot description, URDF)
Before this commit: robot deepracer, 14 links, 13 joints
Links:
- link camera_link_leftcam: geometry visual mesh filename=package://site/meshes/deepracer/camera_link_leftcam.STL
- link camera_link_rightcam: geometry visual mesh filename=package://site/meshes/deepracer/camera_link_rightcam.STL
- link car_body_link_v3: geometry collision mesh filename=package://site/meshes/deepracer/car_body_link_lidar_v3.STL; visual mesh filename=package://site/meshes/deepracer/car_body_link_lidar_v3.STL
- link chassis: geometry visual mesh filename=package://site/meshes/deepracer/chassis.STL
- link laser: geometry collision mesh filename=package://site/meshes/deepracer/laser.STL; visual mesh filename=package://site/meshes/deepracer/laser.STL
- link left_front_wheel: geometry collision mesh filename=package://site/meshes/deepracer/left_front_wheel.STL; visual mesh filename=package://site/meshes/deepracer/left_front_wheel.STL
- link left_rear_wheel: geometry collision mesh filename=package://site/meshes/deepracer/left_rear_wheel.STL; visual mesh filename=package://site/meshes/deepracer/left_rear_wheel.STL
- link left_steering_hinge: geometry visual mesh filename=package://site/meshes/deepracer/left_steering_hinge.STL
- link right_front_wheel: geometry collision mesh filename=package://site/meshes/deepracer/right_front_wheel.STL; visual mesh filename=package://site/meshes/deepracer/right_front_wheel.STL
- link right_rear_wheel: geometry collision mesh filename=package://site/meshes/deepracer/right_rear_wheel.STL; visual mesh filename=package://site/meshes/deepracer/right_rear_wheel.STL
- link right_steering_hinge: geometry visual mesh filename=package://site/meshes/deepracer/right_steering_hinge.STL
- link zed_camera_link_leftcam: geometry visual mesh filename=package://site/meshes/deepracer/zed_camera_link_leftcam.STL
- link zed_camera_link_rightcam: geometry visual mesh filename=package://site/meshes/deepracer/zed_camera_link_rightcam.STL

File: catkin_ws/src/site/urdf/site.urdf.xacro (robot description, xacro)
@@ -110,8 +110,4 @@
   </gazebo>
   <gazebo reference="CPU_4_Link">
-    <material>Gazebo/Black</material>
-    <turnGravityOff>false</turnGravityOff>
-  </gazebo>
-  <gazebo reference="ARS_408_21_2_Link">
     <material>Gazebo/Black</material>
     <turnGravityOff>false</turnGravityOff>
@@ -2270,3 +2266,635 @@
   </joint>
   <!-- deepracer -->
+<link name="chassis">
+    <inertial>
+      <origin
+        xyz="0 0 0"
+        rpy="0 0 0" />
+      <mass
+        value="5.0" />
+      <inertia
+        ixx="0.010609"
+        ixy="0"
+        ixz="0"
+        iyy="0.050409"
+        iyz="0"
+        izz="0.05865" />
+    </inertial>
+    <visual>
+      <origin
+        xyz="0 0 0"
+        rpy="0 0 0" />
+      <geometry>
+        <mesh
+          filename="package://site/meshes/deepracer/chassis.STL" />
+      </geometry>
+    </visual>
+  </link>
+  <joint name="base_link_joint" type="fixed">
+    <origin xyz="0 0 0.023249" rpy="0 0 0" />
+    <parent link="base_link" />
+    <child link="chassis" />
+  </joint>
+  <link
+    name="left_rear_wheel">
+    <inertial>
+      <origin
+        xyz="0 0 0"
+        rpy="0 0 0" />
+      <mass
+        value="0.34055" />
+      <inertia
+        ixx="0.00026046"
+        ixy="0"
+        ixz="0"
+        iyy="0.00041226"
+        iyz="0"
+        izz="0.00026046" />
+    </inertial>
+    <visual>
+      <origin
+        xyz="0 0 0"
+        rpy="0 0 0" />
+      <geometry>
+        <mesh
+          filename="package://site/meshes/deepracer/left_rear_wheel.STL" />
+      </geometry>
+    </visual>
+    <collision>
+      <origin
+        xyz="0 0 0"
+        rpy="0 0 0" />
+      <geometry>
+        <mesh
+          filename="package://site/meshes/deepracer/left_rear_wheel.STL" />
+      </geometry>
+    </collision>
+  </link>
+  <joint
+    name="left_rear_wheel_joint"
+    type="continuous">
+    <origin
+      xyz="-0.081663 0.08105 0.01575"
+      rpy="0 0 0" />
+    <parent
+      link="chassis" />
+    <child
+      link="left_rear_wheel" />
+    <axis
+      xyz="0 1 0" />
+    <limit
+      effort="10"
+      velocity="100" />
+  </joint>
+  <link
+    name="right_rear_wheel">
+    <inertial>
+      <origin
+        xyz="0 0 0"
+        rpy="0 0 0" />
+      <mass
+        value="0.34055" />
+      <inertia
+        ixx="0.00026046"
+        ixy="0"
+        ixz="0"
+        iyy="0.00041226"
+        iyz="0"
+        izz="0.00026046" />
+    </inertial>
+    <visual>
+      <origin
+        xyz="0 0 0"
+        rpy="0 0 0" />
+      <geometry>
+        <mesh
+          filename="package://site/meshes/deepracer/right_rear_wheel.STL" />
+      </geometry>
+    </visual>
+    <collision>
+      <origin
+        xyz="0 0 0"
+        rpy="0 0 0" />
+      <geometry>
+        <mesh
+          filename="package://site/meshes/deepracer/right_rear_wheel.STL" />
+      </geometry>
+    </collision>
+  </link>
+  <joint
+    name="right_rear_wheel_joint"
+    type="continuous">
+    <origin
+      xyz="-0.081663 -0.08105 0.01575"
+      rpy="0 0 0" />
+    <parent
+      link="chassis" />
+    <child
+      link="right_rear_wheel" />
+    <axis
+      xyz="0 1 0" />
+    <limit
+      effort="10"
+      velocity="100" />
+  </joint>
+  <link
+    name="left_steering_hinge">
+    <inertial>
+      <origin
+        xyz="0 0 0"
+        rpy="0 0 0" />
+      <mass
+        value="0.1" />
+      <inertia
+        ixx="4E-06"
+        ixy="0"
+        ixz="0"
+        iyy="4E-06"
+        iyz="0"
+        izz="4E-06" />
+      </inertial>
+    <visual>
+      <origin
+        xyz="0 0 0"
+        rpy="0 0 0" />
+      <geometry>
+        <mesh
+          filename="package://site/meshes/deepracer/left_steering_hinge.STL" />
+      </geometry>
+    </visual>
+  </link>
+  <joint
+    name="left_steering_hinge_joint"
+    type="continuous">
+    <origin
+      xyz="0.082311 0.079601 0.011759"
+      rpy="0 0 0" />
+    <parent
+      link="chassis" />
+    <child
+      link="left_steering_hinge" />
+    <axis
+      xyz="0 0 1" />
+    <limit
+      lower="-1"
+      upper="1"
+      effort="10"
+      velocity="100" />
+  </joint>
+  <link
+    name="left_front_wheel">
+    <inertial>
+      <origin
+        xyz="0 0 0"
+        rpy="0 0 0" />
+      <mass
+        value="0.34055" />
+      <inertia
+        ixx="0.00026046"
+        ixy="0"
+        ixz="0"
+        iyy="0.00041226"
+        iyz="0"
+        izz="0.00026046" />
+    </inertial>
+    <visual>
+      <origin
+        xyz="0 0 0"
+        rpy="0 0 0" />
+      <geometry>
+        <mesh
+          filename="package://site/meshes/deepracer/left_front_wheel.STL" />
+      </geometry>
+    </visual>
+    <collision>
+      <origin
+        xyz="0 0 0"
+        rpy="0 0 0" />
+      <geometry>
+        <mesh
+          filename="package://site/meshes/deepracer/left_front_wheel.STL" />
+      </geometry>
+    </collision>
+  </link>
+  <joint
+    name="left_front_wheel_joint"
+    type="continuous">
+    <origin
+      xyz="0 0 0"
+      rpy="0 0 0" />
+    <parent
+      link="left_steering_hinge" />
+    <child
+      link="left_front_wheel" />
+    <axis
+      xyz="0 1 0" />
+    <limit
+      effort="10"
+      velocity="100" />
+  </joint>
+  <link
+    name="right_steering_hinge">
+    <inertial>
+      <origin
+        xyz="0 0 0"
+        rpy="0 0 0" />
+      <mass
+        value="0.1" />
+      <inertia
+        ixx="4E-06"
+        ixy="0"
+        ixz="0"
+        iyy="4E-06"
+        iyz="0"
+        izz="4E-06" />
+    </inertial>
+    <visual>
+      <origin
+        xyz="0 0 0"
+        rpy="0 0 0" />
+      <geometry>
+        <mesh
+          filename="package://site/meshes/deepracer/right_steering_hinge.STL" />
+      </geometry>
+    </visual>
+  </link>
+  <joint
+    name="right_steering_hinge_joint"
+    type="continuous">
+    <origin
+      xyz="0.082311 -0.079601 0.011759"
+      rpy="0 0 0" />
+    <parent
+      link="chassis" />
+    <child
+      link="right_steering_hinge" />
+    <axis
+      xyz="0 0 1" />
+    <limit
+      lower="-1"
+      upper="1"
+      effort="10"
+      velocity="100" />
+  </joint>
+  <link
+    name="right_front_wheel">
+    <inertial>
+      <origin
+        xyz="0 0 0"
+        rpy="0 0 0" />
+      <mass
+        value="0.34055" />
+      <inertia
+        ixx="0.00026046"
+        ixy="0"
+        ixz="0"
+        iyy="0.00041226"
+        iyz="0"
+        izz="0.00026046" />
+    </inertial>
+    <visual>
+      <origin
+        xyz="0 0 0"
+        rpy="0 0 0" />
+      <geometry>
+        <mesh
+          filename="package://site/meshes/deepracer/right_front_wheel.STL" />
+      </geometry>
+    </visual>
+    <collision>
+      <origin
+        xyz="0 0 0"
+        rpy="0 0 0" />
+      <geometry>
+        <mesh
+          filename="package://site/meshes/deepracer/right_front_wheel.STL" />
+      </geometry>
+    </collision>
+  </link>
+  <joint
+    name="right_front_wheel_joint"
+    type="continuous">
+    <origin
+      xyz="0 0 0"
+      rpy="0 0 0" />
+    <parent
+      link="right_steering_hinge" />
+    <child
+      link="right_front_wheel" />
+    <axis
+      xyz="0 1 0" />
+    <limit
+      effort="10"
+      velocity="100" />
+  </joint>
+  <link
+    name="zed_camera_link_leftcam">
+    <inertial>
+      <origin
+        xyz="0.019881 6.2875E-05 0.034966"
+        rpy="0 0 0" />
+      <mass
+        value="1e-3" />
+      <inertia
+        ixx="1e-6"
+        ixy="0"
+        ixz="0"
+        iyy="1e-6"
+        iyz="0"
+        izz="1e-6" />
+    </inertial>
+    <visual>
+      <origin
+        xyz="0 0 0"
+        rpy="0 0 0" />
+      <geometry>
+        <mesh
+          filename="package://site/meshes/deepracer/zed_camera_link_leftcam.STL" />
+      </geometry>
+    </visual>
+  </link>
+  <joint
+    name="zed_camera_joint_leftcam"
+    type="fixed">
+    <origin
+      xyz="0.091711 0.03 0.080023"
+      rpy="0 0.2618 0" />
+    <parent
+      link="chassis" />
+    <child
+      link="zed_camera_link_leftcam" />
+    <axis
+      xyz="0 0 0" />
+  </joint>
+  <link
+    name="camera_link_leftcam">
+    <inertial>
+      <origin
+        xyz="0.0005 0 0"
+        rpy="0 0 0" />
+      <mass
+        value="1e-3" />
+      <inertia
+        ixx="1e-6"
+        ixy="0"
+        ixz="0"
+        iyy="1e-6"
+        iyz="0"
+        izz="1e-6" />
+    </inertial>
+  <visual>
+      <origin
+        xyz="0 0 0"
+        rpy="0 0 0" />
+      <geometry>
+        <mesh
+          filename="package://site/meshes/deepracer/camera_link_leftcam.STL" />
+      </geometry>
+    </visual>
+  </link>
+  <joint
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