Commit message: add new site

File: catkin_ws/src/ARS_gazebo_plugin/radar_plugin/urdf/ARS_408_21_2.urdf.xacro (robot description, xacro)
@@ -38,5 +38,5 @@
             </collision>
             <inertial>
-                <origin xyz="0.00168514324992164 0.0154191890257049 -2.61569096045022E-05" rpy="0 0 0" />
+                <origin xyz="0.00168514324992186 0.0154191890257047 -2.61569096043912E-05" rpy="0 0 0" />
                 <mass value="3.09545763589521"/>
                 <inertia
