Commit message: update deepracer

File: ROS_WS/site_ws/src/site_model/urdf/deepracer.urdf (robot description, URDF)
Before this commit: robot deepracer, 14 links, 13 joints
Links:
- link camera_link_rightcam: geometry visual mesh filename=package://pkg/meshes/deepracer/camera_link_rightcam.STL
- link car_body_link_v3: geometry collision mesh filename=package://pkg/meshes/deepracer/car_body_link_lidar_v3.STL; visual mesh filename=package://pkg/meshes/deepracer/car_body_link_lidar_v3.STL
- link chassis: geometry visual mesh filename=package://pkg/meshes/deepracer/chassis.STL
- link laser: geometry collision mesh filename=package://pkg/meshes/deepracer/laser.STL; visual mesh filename=package://pkg/meshes/deepracer/laser.STL
- link left_front_wheel: geometry collision mesh filename=package://pkg/meshes/deepracer/left_front_wheel.STL; visual mesh filename=package://pkg/meshes/deepracer/left_front_wheel.STL
- link left_rear_wheel: geometry collision mesh filename=package://pkg/meshes/deepracer/left_rear_wheel.STL; visual mesh filename=package://pkg/meshes/deepracer/left_rear_wheel.STL
- link left_steering_hinge: geometry visual mesh filename=package://pkg/meshes/deepracer/left_steering_hinge.STL
- link right_front_wheel: geometry collision mesh filename=package://pkg/meshes/deepracer/right_front_wheel.STL; visual mesh filename=package://pkg/meshes/deepracer/right_front_wheel.STL
- link right_rear_wheel: geometry collision mesh filename=package://pkg/meshes/deepracer/right_rear_wheel.STL; visual mesh filename=package://pkg/meshes/deepracer/right_rear_wheel.STL
- link right_steering_hinge: geometry visual mesh filename=package://pkg/meshes/deepracer/right_steering_hinge.STL
- link zed_camera_link_leftcam: geometry visual mesh filename=package://pkg/meshes/deepracer/zed_camera_link_leftcam.STL
- link zed_camera_link_rightcam: geometry visual mesh filename=package://pkg/meshes/deepracer/zed_camera_link_rightcam.STL
Joints:
- joint left_steering_hinge_joint: type fixed -> continuous
- joint right_steering_hinge_joint: type fixed -> continuous

File: ROS_WS/site_ws/src/site_model/urdf/deepracer.xacro (robot description, xacro)
@@ -1,9 +1,12 @@
-<?xml version="1.0"?>
+<?xml version="1.0" encoding="utf-8"?>
 <!-- This URDF was automatically created by SolidWorks to URDF Exporter! Originally created by Stephen Brawner (brawner@gmail.com)
      Commit Version: 1.5.1-0-g916b5db  Build Version: 1.5.7152.31018
      For more information, please see http://wiki.ros.org/sw_urdf_exporter -->
-<robot xmlns:xacro="http://www.ros.org/wiki/xacro" name="deepracer">
-<xacro:macro name="deepracer" params="parent:=base_link name:=deepracer">
+<robot name="deepracer">
 <!-- Links and Joints -->
+  <link name="base_link" />
+<gazebo reference="base_link">
+    <pose>0 0 0 0 0 0</pose>
+</gazebo>
   <link name="chassis">
     <inertial>
@@ -27,5 +30,5 @@
       <geometry>
         <mesh
-          filename="package://site_model/meshes/deepracer/chassis.STL" />
+          filename="package://pkg/meshes/deepracer/chassis.STL" />
       </geometry>
     </visual>
@@ -58,5 +61,5 @@
       <geometry>
         <mesh
-          filename="package://site_model/meshes/deepracer/left_rear_wheel.STL" />
+          filename="package://pkg/meshes/deepracer/left_rear_wheel.STL" />
       </geometry>
     </visual>
@@ -67,5 +70,5 @@
       <geometry>
         <mesh
-          filename="package://site_model/meshes/deepracer/left_rear_wheel.STL" />
+          filename="package://pkg/meshes/deepracer/left_rear_wheel.STL" />
       </geometry>
     </collision>
@@ -87,4 +90,16 @@
       velocity="100" />
   </joint>
+  <transmission name="left_rear_axle_trans">
+      <type>transmission_interface/SimpleTransmission</type>
+      <joint name="left_rear_wheel_joint">
+        <hardwareInterface>hardware_interface/EffortJointInterface</hardwareInterface>
+      </joint>
+      <actuator name="left_rear_axle_act">
+        <!-- This hardwareInterface element exists for compatibility
+             with ROS Hydro. -->
+        <hardwareInterface>hardware_interface/EffortJointInterface</hardwareInterface>
+        <mechanicalReduction>1</mechanicalReduction>
+      </actuator>
+  </transmission>
   <link
     name="right_rear_wheel">
@@ -109,5 +124,5 @@
       <geometry>
         <mesh
-          filename="package://site_model/meshes/deepracer/right_rear_wheel.STL" />
+          filename="package://pkg/meshes/deepracer/right_rear_wheel.STL" />
       </geometry>
     </visual>
@@ -118,5 +133,5 @@
       <geometry>
         <mesh
-          filename="package://site_model/meshes/deepracer/right_rear_wheel.STL" />
+          filename="package://pkg/meshes/deepracer/right_rear_wheel.STL" />
       </geometry>
     </collision>
@@ -138,4 +153,16 @@
       velocity="100" />
   </joint>
+    <transmission name="right_rear_axle_trans">
+      <type>transmission_interface/SimpleTransmission</type>
+      <joint name="right_rear_wheel_joint">
+        <hardwareInterface>hardware_interface/EffortJointInterface</hardwareInterface>
+      </joint>
+      <actuator name="right_rear_axle_act">
+        <!-- This hardwareInterface element exists for compatibility
+             with ROS Hydro. -->
+        <hardwareInterface>hardware_interface/EffortJointInterface</hardwareInterface>
+        <mechanicalReduction>1</mechanicalReduction>
+      </actuator>
+  </transmission>
   <link
     name="left_steering_hinge">
@@ -160,5 +187,5 @@
       <geometry>
         <mesh
-          filename="package://site_model/meshes/deepracer/left_steering_hinge.STL" />
+          filename="package://pkg/meshes/deepracer/left_steering_hinge.STL" />
       </geometry>
     </visual>
@@ -166,5 +193,5 @@
   <joint
     name="left_steering_hinge_joint"
-    type="fixed">
+    type="continuous">
     <origin
       xyz="0.082311 0.079601 0.011759"
@@ -182,4 +209,16 @@
       velocity="100" />
   </joint>
+  <transmission name="left_steering_trans">
+      <type>transmission_interface/SimpleTransmission</type>
+      <joint name="left_steering_hinge_joint">
+        <hardwareInterface>hardware_interface/EffortJointInterface</hardwareInterface>
+      </joint>
+      <actuator name="left_steering_act">
+        <!-- This hardwareInterface element exists for compatibility
+             with ROS Hydro. -->
+        <hardwareInterface>hardware_interface/EffortJointInterface</hardwareInterface>
+        <mechanicalReduction>1</mechanicalReduction>
+      </actuator>
+  </transmission>
   <link
     name="left_front_wheel">
@@ -204,5 +243,5 @@
       <geometry>
         <mesh
-          filename="package://site_model/meshes/deepracer/left_front_wheel.STL" />
+          filename="package://pkg/meshes/deepracer/left_front_wheel.STL" />
       </geometry>
     </visual>
@@ -213,5 +252,5 @@
       <geometry>
         <mesh
-          filename="package://site_model/meshes/deepracer/left_front_wheel.STL" />
+          filename="package://pkg/meshes/deepracer/left_front_wheel.STL" />
       </geometry>
     </collision>
@@ -233,4 +272,16 @@
       velocity="100" />
   </joint>
+  <transmission name="left_front_axle_trans">
+      <type>transmission_interface/SimpleTransmission</type>
+      <joint name="left_front_wheel_joint">
+        <hardwareInterface>hardware_interface/EffortJointInterface</hardwareInterface>
+      </joint>
+      <actuator name="left_front_axle_act">
+        <!-- This hardwareInterface element exists for compatibility
+             with ROS Hydro. -->
+        <hardwareInterface>hardware_interface/EffortJointInterface</hardwareInterface>
+        <mechanicalReduction>1</mechanicalReduction>
+      </actuator>
+  </transmission>
   <link
     name="right_steering_hinge">
@@ -255,5 +306,5 @@
       <geometry>
         <mesh
-          filename="package://site_model/meshes/deepracer/right_steering_hinge.STL" />
+          filename="package://pkg/meshes/deepracer/right_steering_hinge.STL" />
       </geometry>
     </visual>
@@ -261,5 +312,5 @@
   <joint
     name="right_steering_hinge_joint"
-    type="fixed">
+    type="continuous">
     <origin
       xyz="0.082311 -0.079601 0.011759"
@@ -277,4 +328,16 @@
       velocity="100" />
   </joint>
+  <transmission name="right_steering_trans">
+      <type>transmission_interface/SimpleTransmission</type>
+      <joint name="right_steering_hinge_joint">
+        <hardwareInterface>hardware_interface/EffortJointInterface</hardwareInterface>
+      </joint>
+      <actuator name="right_steering_act">
+        <!-- This hardwareInterface element exists for compatibility
+             with ROS Hydro. -->
+        <hardwareInterface>hardware_interface/EffortJointInterface</hardwareInterface>
+        <mechanicalReduction>1</mechanicalReduction>
+      </actuator>
+  </transmission>
   <link
     name="right_front_wheel">
@@ -299,5 +362,5 @@
       <geometry>
         <mesh
-          filename="package://site_model/meshes/deepracer/right_front_wheel.STL" />
+          filename="package://pkg/meshes/deepracer/right_front_wheel.STL" />
       </geometry>
     </visual>
@@ -308,5 +371,5 @@
       <geometry>
         <mesh
-          filename="package://site_model/meshes/deepracer/right_front_wheel.STL" />
+          filename="package://pkg/meshes/deepracer/right_front_wheel.STL" />
       </geometry>
     </collision>
@@ -328,4 +391,16 @@
       velocity="100" />
   </joint>
+    <transmission name="right_front_axle_trans">
+      <type>transmission_interface/SimpleTransmission</type>
+      <joint name="right_front_wheel_joint">
+        <hardwareInterface>hardware_interface/EffortJointInterface</hardwareInterface>
+      </joint>
+      <actuator name="right_front_axle_act">
+        <!-- This hardwareInterface element exists for compatibility
+             with ROS Hydro. -->
+        <hardwareInterface>hardware_interface/EffortJointInterface</hardwareInterface>
+        <mechanicalReduction>1</mechanicalReduction>
+      </actuator>
+  </transmission>
   <link
     name="zed_camera_link_leftcam">
@@ -350,5 +425,5 @@
       <geometry>
         <mesh
-          filename="package://site_model/meshes/deepracer/zed_camera_link_leftcam.STL" />
+          filename="package://pkg/meshes/deepracer/zed_camera_link_leftcam.STL" />
       </geometry>
     </visual>
@@ -389,5 +464,5 @@
       <geometry>
         <mesh
-          filename="package://site_model/meshes/deepracer/camera_link_leftcam.STL" />
+          filename="package://pkg/meshes/deepracer/camera_link_leftcam.STL" />
       </geometry>
     </visual> -->
@@ -428,5 +503,5 @@
       <geometry>
         <mesh
-          filename="package://site_model/meshes/deepracer/zed_camera_link_rightcam.STL" />
+          filename="package://pkg/meshes/deepracer/zed_camera_link_rightcam.STL" />
       </geometry>
     </visual>
@@ -461,13 +536,13 @@
         izz="1e-6" />
     </inertial>
-<!--     <visual>
-      <origin
-        xyz="0 0 0"
-        rpy="0 0 0" />
-      <geometry>
-        <mesh
-          filename="package://site_model/meshes/deepracer/camera_link_rightcam.STL" />
-      </geometry>
-    </visual> -->
+    <visual>
+      <origin
+        xyz="0 0 0"
+        rpy="0 0 0" />
+      <geometry>
+        <mesh
+          filename="package://pkg/meshes/deepracer/camera_link_rightcam.STL" />
+      </geometry>
+    </visual>
   </link>
   <joint
@@ -506,5 +581,5 @@
       <geometry>
         <mesh
-          filename="package://site_model/meshes/deepracer/laser.STL" />
+          filename="package://pkg/meshes/deepracer/laser.STL" />
       </geometry>
     </visual>
@@ -515,5 +590,5 @@
       <geometry>
         <mesh
-          filename="package://site_model/meshes/deepracer/laser.STL" />
+          filename="package://pkg/meshes/deepracer/laser.STL" />
       </geometry>
     </collision>
@@ -524,5 +599,5 @@
     <origin
       xyz="0.02913 0 0.16145"
-      rpy="0 0 3.1416" />
+      rpy="0 0 0" />
     <parent
       link="chassis" />
@@ -554,5 +629,5 @@
       <geometry>
         <mesh
-          filename="package://site_model/meshes/deepracer/car_body_link_lidar_v3.STL" />
+          filename="package://pkg/meshes/deepracer/car_body_link_lidar_v3.STL" />
       </geometry>
     </visual>
@@ -563,5 +638,5 @@
       <geometry>
         <mesh
-          filename="package://site_model/meshes/deepracer/car_body_link_lidar_v3.STL" />
+          filename="package://pkg/meshes/deepracer/car_body_link_lidar_v3.STL" />
       </geometry>
     </collision>
@@ -583,4 +658,5 @@
 <!-- Vehicle body -->
   <gazebo reference = "chassis">
+<pose>0 0 0 0 0 0</pose>
    <material>Gazebo/Grey</material>
    <mu1 value="0.0"/>
@@ -589,52 +665,61 @@
   </gazebo>
   <gazebo reference = "left_rear_wheel">
+<pose>0 0 0 0 0 0</pose>
    <material>Gazebo/DarkGrey</material>
-   <mu1 value="0.5"/>
-   <mu2 value="0.5"/>
+   <mu1 value="500"/>
+   <mu2 value="500"/>
    <kp  value="1000000.0" />
-   <kd  value="1.0" />
+   <kd  value="100000.0" />
    <fdir1 value="1 0 0"/>
   </gazebo>
   <gazebo reference = "left_front_wheel">
+<pose>0 0 0 0 0 0</pose>
    <material>Gazebo/DarkGrey</material>
-   <mu1 value="0.5"/>
-   <mu2 value="0.5"/>
+   <mu1 value="500"/>
+   <mu2 value="500"/>
    <kp  value="1000000.0" />
-   <kd  value="1.0" />
+   <kd  value="100000.0" />
    <fdir1 value="1 0 0"/>
   </gazebo>
   <gazebo reference = "right_rear_wheel">
+<pose>0 0 0 0 0 0</pose>
    <material>Gazebo/DarkGrey</material>
-   <mu1 value="0.5"/>
-   <mu2 value="0.5"/>
+   <mu1 value="500"/>
+   <mu2 value="500"/>
    <kp  value="1000000.0" />
-   <kd  value="1.0" />
+   <kd  value="100000.0" />
    <fdir1 value="1 0 0"/>
   </gazebo>
   <gazebo reference = "right_front_wheel">
+<pose>0 0 0 0 0 0</pose>
    <material>Gazebo/DarkGrey</material>
-   <mu1 value="0.5"/>
-   <mu2 value="0.5"/>
+   <mu1 value="500"/>
+   <mu2 value="500"/>
    <kp  value="1000000.0" />
-   <kd  value="1.0" />
+   <kd  value="100000.0" />
    <fdir1 value="1 0 0"/>
   </gazebo>
   <gazebo reference = "left_steering_hinge">
+<pose>0 0 0 0 0 0</pose>
    <material>Gazebo/DarkGrey</material>
   </gazebo>
   <gazebo reference = "right_steering_hinge">
+<pose>0 0 0 0 0 0</pose>
    <material>Gazebo/DarkGrey</material>
   </gazebo>
   <gazebo reference = "zed_camera_link_leftcam">
+<pose>0 0 0 0 0 0</pose>
    <material>Gazebo/DarkGrey</material>
   </gazebo>
   <gazebo reference = "zed_camera_link_rightcam">
+<pose>0 0 0 0 0 0</pose>
    <material>Gazebo/DarkGrey</material>
   </gazebo>
   <gazebo reference = "car_body_link_v3">
+<pose>0 0 0 0 0 0</pose>
    <material>Gazebo/Grey</material>
   </gazebo>
 <!-- Chassis Controller-->
-   <gazebo>
+   <!--gazebo>
     <plugin name="skid_steer_drive_controller" filename="libgazebo_ros_skid_steer_drive.so">
       <updateRate>30</updateRate>
@@ -651,8 +736,15 @@
       <odometryTopic>odom</odometryTopic>
       <odometryFrame>odom</odometryFrame>
-      <covariance_x>0.0001</covariance_x>
-      <covariance_y>0.0001</covariance_y>
-      <covariance_yaw>0.0001</covariance_yaw>
+      <covariance_x>0</covariance_x>
+      <covariance_y>0</covariance_y>
+      <covariance_yaw>0</covariance_yaw>
       <broadcastTF>true</broadcastTF>
+    </plugin>
+  </gazebo-->
+  <gazebo>
+    <plugin name="gazebo_ros_control" filename="libgazebo_ros_control.so">
+    <legacyModeNS>true</legacyModeNS>
+    <robotSimType>gazebo_ros_control/DefaultRobotHWSim</robotSimType>
+    <robotNamespace>$(arg bodyframe)</robotNamespace>
     </plugin>
   </gazebo>
@@ -732,5 +824,5 @@
       <pose>0 0 0 0 0 0</pose>
       <visualize>false</visualize>
-      <update_rate>30</update_rate>
+      <update_rate>10</update_rate>
       <ray>
         <scan>
@@ -738,6 +830,8 @@
             <samples>600</samples>
             <resolution>1</resolution>
-            <min_angle>-2.61799</min_angle>
-            <max_angle>2.61799</max_angle>
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
Commit message: add pkg

File: ROS_WS/site_ws/src/site_model/urdf/deepracer.urdf (robot description, URDF)
Before this commit: robot deepracer, 14 links, 13 joints
Links:
- link camera_link_rightcam: geometry visual mesh filename=package://site_model/meshes/deepracer/camera_link_rightcam.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
- link car_body_link_v3: geometry collision mesh filename=package://site_model/meshes/deepracer/car_body_link_lidar_v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; visual mesh filename=package://site_model/meshes/deepracer/car_body_link_lidar_v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
- link chassis: geometry visual mesh filename=package://site_model/meshes/deepracer/chassis.STL
- link laser: geometry collision mesh filename=package://site_model/meshes/deepracer/laser.STL; visual mesh filename=package://site_model/meshes/deepracer/laser.STL
- link left_front_wheel: geometry collision mesh filename=package://site_model/meshes/deepracer/left_front_wheel.STL; visual mesh filename=package://site_model/meshes/deepracer/left_front_wheel.STL
- link left_rear_wheel: geometry collision mesh filename=package://site_model/meshes/deepracer/left_rear_wheel.STL; visual mesh filename=package://site_model/meshes/deepracer/left_rear_wheel.STL
- link left_steering_hinge: geometry visual mesh filename=package://site_model/meshes/deepracer/left_steering_hinge.S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
- link right_front_wheel: geometry collision mesh filename=package://site_model/meshes/deepracer/right_front_wheel.STL; visual mesh filename=package://site_model/meshes/deepracer/right_front_wheel.STL
- link right_rear_wheel: geometry collision mesh filename=package://site_model/meshes/deepracer/right_rear_wheel.STL; visual mesh filename=package://site_model/meshes/deepracer/right_rear_wheel.STL
- link right_steering_hinge: geometry visual mesh filename=package://site_model/meshes/deepracer/right_steering_hinge.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
- link zed_camera_link_leftcam: geometry visual mesh filename=package://site_model/meshes/deepracer/zed_camera_link_leftc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
- link zed_camera_link_rightcam: geometry visual mesh filename=package://site_model/meshes/deepracer/zed_camera_link_right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
