Commit message: update all

File: site_ws/src/site_model/urdf/deepracer.urdf (robot description, URDF)
Before this commit: robot deepracer, 14 links, 13 joints
Joints:
- joint left_steering_hinge_joint: type fixed -> continuous
- joint right_steering_hinge_joint: type fixed -> continuous

File: site_ws/src/site_model/urdf/site_model.urdf.xacro (robot description, xacro)
@@ -161,5 +161,5 @@
 <!-- Lidar11 points1 -->
   <joint name="velodyne11_base_mount_joint" type="fixed">
-    <origin rpy="-1.570796327 0 0" xyz="0 -0.475 -0.2"/>
+    <origin rpy="-1.570796327 -0.7853981634 0" xyz="0 -0.475 -0.2"/>
     <parent link="pole1_Link"/>
     <child link="velodyne11_base_link"/>
@@ -243,5 +243,5 @@
         <min_range>0.9</min_range>
         <max_range>130.0</max_range>
-        <gaussianNoise>0.008</gaussianNoise>
+        <gaussianNoise>0.006</gaussianNoise>
       </plugin>
     </sensor>
@@ -249,5 +249,5 @@
   <!-- Lidar12 points 2-->
   <joint name="velodyne12_base_mount_joint" type="fixed">
-    <origin rpy="-1.570796327 0 0" xyz="0 -0.475 1.2"/>
+    <origin rpy="-1.570796327 -0.7853981634 0" xyz="0 -0.475 1.2"/>
     <parent link="pole1_Link"/>
     <child link="velodyne12_base_link"/>
@@ -331,5 +331,5 @@
         <min_range>0.9</min_range>
         <max_range>130.0</max_range>
-        <gaussianNoise>0.008</gaussianNoise>
+        <gaussianNoise>0.006</gaussianNoise>
       </plugin>
     </sensor>
@@ -1258,5 +1258,5 @@
   <!-- Lidar_2 points3 -->
   <joint name="velodyne2_base_mount_joint" type="fixed">
-    <origin rpy="-1.570796327 0 0" xyz="0 -0.26 1.14"/>
+    <origin rpy="-1.570796327 0 0" xyz="0 -0.38 1.14"/>
     <parent link="pole4_Link"/>
     <child link="velodyne2_base_link"/>
@@ -1340,5 +1340,5 @@
         <min_range>0.9</min_range>
         <max_range>130.0</max_range>
-        <gaussianNoise>0.008</gaussianNoise>
+        <gaussianNoise>0.006</gaussianNoise>
       </plugin>
     </sensor>
