Commit message: update pkg

File: src/pkg/urdf/deepracer.xacro (robot description, xacro)
@@ -6,4 +6,7 @@
 <!-- Links and Joints -->
   <link name="base_link" />
+<gazebo reference="base_link">
+    <pose>0 0 0 0 0 0</pose>
+</gazebo>
   <link name="chassis">
     <inertial>
@@ -87,4 +90,16 @@
       velocity="100" />
   </joint>
+  <transmission name="left_rear_axle_trans">
+      <type>transmission_interface/SimpleTransmission</type>
+      <joint name="left_rear_wheel_joint">
+        <hardwareInterface>hardware_interface/EffortJointInterface</hardwareInterface>
+      </joint>
+      <actuator name="left_rear_axle_act">
+        <!-- This hardwareInterface element exists for compatibility
+             with ROS Hydro. -->
+        <hardwareInterface>hardware_interface/EffortJointInterface</hardwareInterface>
+        <mechanicalReduction>1</mechanicalReduction>
+      </actuator>
+  </transmission>
   <link
     name="right_rear_wheel">
@@ -138,4 +153,16 @@
       velocity="100" />
   </joint>
+    <transmission name="right_rear_axle_trans">
+      <type>transmission_interface/SimpleTransmission</type>
+      <joint name="right_rear_wheel_joint">
+        <hardwareInterface>hardware_interface/EffortJointInterface</hardwareInterface>
+      </joint>
+      <actuator name="right_rear_axle_act">
+        <!-- This hardwareInterface element exists for compatibility
+             with ROS Hydro. -->
+        <hardwareInterface>hardware_interface/EffortJointInterface</hardwareInterface>
+        <mechanicalReduction>1</mechanicalReduction>
+      </actuator>
+  </transmission>
   <link
     name="left_steering_hinge">
@@ -166,5 +193,5 @@
   <joint
     name="left_steering_hinge_joint"
-    type="fixed">
+    type="continuous">
     <origin
       xyz="0.082311 0.079601 0.011759"
@@ -182,4 +209,16 @@
       velocity="100" />
   </joint>
+  <transmission name="left_steering_trans">
+      <type>transmission_interface/SimpleTransmission</type>
+      <joint name="left_steering_hinge_joint">
+        <hardwareInterface>hardware_interface/EffortJointInterface</hardwareInterface>
+      </joint>
+      <actuator name="left_steering_act">
+        <!-- This hardwareInterface element exists for compatibility
+             with ROS Hydro. -->
+        <hardwareInterface>hardware_interface/EffortJointInterface</hardwareInterface>
+        <mechanicalReduction>1</mechanicalReduction>
+      </actuator>
+  </transmission>
   <link
     name="left_front_wheel">
@@ -233,4 +272,16 @@
       velocity="100" />
   </joint>
+  <transmission name="left_front_axle_trans">
+      <type>transmission_interface/SimpleTransmission</type>
+      <joint name="left_front_wheel_joint">
+        <hardwareInterface>hardware_interface/EffortJointInterface</hardwareInterface>
+      </joint>
+      <actuator name="left_front_axle_act">
+        <!-- This hardwareInterface element exists for compatibility
+             with ROS Hydro. -->
+        <hardwareInterface>hardware_interface/EffortJointInterface</hardwareInterface>
+        <mechanicalReduction>1</mechanicalReduction>
+      </actuator>
+  </transmission>
   <link
     name="right_steering_hinge">
@@ -261,5 +312,5 @@
   <joint
     name="right_steering_hinge_joint"
-    type="fixed">
+    type="continuous">
     <origin
       xyz="0.082311 -0.079601 0.011759"
@@ -277,4 +328,16 @@
       velocity="100" />
   </joint>
+  <transmission name="right_steering_trans">
+      <type>transmission_interface/SimpleTransmission</type>
+      <joint name="right_steering_hinge_joint">
+        <hardwareInterface>hardware_interface/EffortJointInterface</hardwareInterface>
+      </joint>
+      <actuator name="right_steering_act">
+        <!-- This hardwareInterface element exists for compatibility
+             with ROS Hydro. -->
+        <hardwareInterface>hardware_interface/EffortJointInterface</hardwareInterface>
+        <mechanicalReduction>1</mechanicalReduction>
+      </actuator>
+  </transmission>
   <link
     name="right_front_wheel">
@@ -328,4 +391,16 @@
       velocity="100" />
   </joint>
+    <transmission name="right_front_axle_trans">
+      <type>transmission_interface/SimpleTransmission</type>
+      <joint name="right_front_wheel_joint">
+        <hardwareInterface>hardware_interface/EffortJointInterface</hardwareInterface>
+      </joint>
+      <actuator name="right_front_axle_act">
+        <!-- This hardwareInterface element exists for compatibility
+             with ROS Hydro. -->
+        <hardwareInterface>hardware_interface/EffortJointInterface</hardwareInterface>
+        <mechanicalReduction>1</mechanicalReduction>
+      </actuator>
+  </transmission>
   <link
     name="zed_camera_link_leftcam">
@@ -461,5 +536,5 @@
         izz="1e-6" />
     </inertial>
-<!--     <visual>
+    <visual>
       <origin
         xyz="0 0 0"
@@ -469,5 +544,5 @@
           filename="package://pkg/meshes/deepracer/camera_link_rightcam.STL" />
       </geometry>
-    </visual> -->
+    </visual>
   </link>
   <joint
@@ -524,5 +599,5 @@
     <origin
       xyz="0.02913 0 0.16145"
-      rpy="0 0 3.1416" />
+      rpy="0 0 0" />
     <parent
       link="chassis" />
@@ -583,4 +658,5 @@
 <!-- Vehicle body -->
   <gazebo reference = "chassis">
+<pose>0 0 0 0 0 0</pose>
    <material>Gazebo/Grey</material>
    <mu1 value="0.0"/>
@@ -589,55 +665,64 @@
   </gazebo>
   <gazebo reference = "left_rear_wheel">
+<pose>0 0 0 0 0 0</pose>
    <material>Gazebo/DarkGrey</material>
-   <mu1 value="0.5"/>
-   <mu2 value="0.5"/>
+   <mu1 value="500"/>
+   <mu2 value="500"/>
    <kp  value="1000000.0" />
-   <kd  value="1.0" />
+   <kd  value="100000.0" />
    <fdir1 value="1 0 0"/>
   </gazebo>
   <gazebo reference = "left_front_wheel">
+<pose>0 0 0 0 0 0</pose>
    <material>Gazebo/DarkGrey</material>
-   <mu1 value="0.5"/>
-   <mu2 value="0.5"/>
+   <mu1 value="500"/>
+   <mu2 value="500"/>
    <kp  value="1000000.0" />
-   <kd  value="1.0" />
+   <kd  value="100000.0" />
    <fdir1 value="1 0 0"/>
   </gazebo>
   <gazebo reference = "right_rear_wheel">
+<pose>0 0 0 0 0 0</pose>
    <material>Gazebo/DarkGrey</material>
-   <mu1 value="0.5"/>
-   <mu2 value="0.5"/>
+   <mu1 value="500"/>
+   <mu2 value="500"/>
    <kp  value="1000000.0" />
-   <kd  value="1.0" />
+   <kd  value="100000.0" />
    <fdir1 value="1 0 0"/>
   </gazebo>
   <gazebo reference = "right_front_wheel">
+<pose>0 0 0 0 0 0</pose>
    <material>Gazebo/DarkGrey</material>
-   <mu1 value="0.5"/>
-   <mu2 value="0.5"/>
+   <mu1 value="500"/>
+   <mu2 value="500"/>
    <kp  value="1000000.0" />
-   <kd  value="1.0" />
+   <kd  value="100000.0" />
    <fdir1 value="1 0 0"/>
   </gazebo>
   <gazebo reference = "left_steering_hinge">
+<pose>0 0 0 0 0 0</pose>
    <material>Gazebo/DarkGrey</material>
   </gazebo>
   <gazebo reference = "right_steering_hinge">
+<pose>0 0 0 0 0 0</pose>
    <material>Gazebo/DarkGrey</material>
   </gazebo>
   <gazebo reference = "zed_camera_link_leftcam">
+<pose>0 0 0 0 0 0</pose>
    <material>Gazebo/DarkGrey</material>
   </gazebo>
   <gazebo reference = "zed_camera_link_rightcam">
+<pose>0 0 0 0 0 0</pose>
    <material>Gazebo/DarkGrey</material>
   </gazebo>
   <gazebo reference = "car_body_link_v3">
+<pose>0 0 0 0 0 0</pose>
    <material>Gazebo/Grey</material>
   </gazebo>
 <!-- Chassis Controller-->
-   <gazebo>
+   <!--gazebo>
     <plugin name="skid_steer_drive_controller" filename="libgazebo_ros_skid_steer_drive.so">
       <updateRate>30</updateRate>
-      <robotNamespace>$(arg bodyframe)</robotNamespace>
+      <robotNamespace>/</robotNamespace>
       <leftFrontJoint>left_front_wheel_joint</leftFrontJoint>
       <rightFrontJoint>right_front_wheel_joint</rightFrontJoint>
@@ -646,13 +731,20 @@
       <wheelSeparation>0.159202</wheelSeparation>
       <wheelDiameter>0.06</wheelDiameter>
-      <robotBaseFrame>$(arg bodyframe)/base_link</robotBaseFrame>
+      <robotBaseFrame>base_link</robotBaseFrame>
       <torque>20</torque>
       <commandTopic>cmd_vel</commandTopic>
       <odometryTopic>odom</odometryTopic>
       <odometryFrame>odom</odometryFrame>
-      <covariance_x>0.0001</covariance_x>
-      <covariance_y>0.0001</covariance_y>
-      <covariance_yaw>0.0001</covariance_yaw>
+      <covariance_x>0</covariance_x>
+      <covariance_y>0</covariance_y>
+      <covariance_yaw>0</covariance_yaw>
       <broadcastTF>true</broadcastTF>
+    </plugin>
+  </gazebo-->
+  <gazebo>
+    <plugin name="gazebo_ros_control" filename="libgazebo_ros_control.so">
+    <legacyModeNS>true</legacyModeNS>
+    <robotSimType>gazebo_ros_control/DefaultRobotHWSim</robotSimType>
+    <robotNamespace>$(arg bodyframe)</robotNamespace>
     </plugin>
   </gazebo>
@@ -732,5 +824,5 @@
       <pose>0 0 0 0 0 0</pose>
       <visualize>false</visualize>
-      <update_rate>30</update_rate>
+      <update_rate>10</update_rate>
       <ray>
         <scan>
@@ -738,6 +830,8 @@
             <samples>600</samples>
             <resolution>1</resolution>
-            <min_angle>-2.61799</min_angle>
-            <max_angle>2.61799</max_angle>
+             <min_angle>-3.1415926</min_angle>
+             <max_angle>3.1415926</max_angle>
+            <!--min_angle>0.52351</min_angle>
+            <max_angle>5.75949</max_angle-->
           </horizontal>
         </scan>
@@ -749,14 +843,13 @@
         <noise>
           <mean>0.0</mean>
-          <stddev>0.01</stddev>
+          <stddev>0</stddev>
         </noise>
       </ray>
        <plugin name="rp_lidar" filename="libgazebo_ros_laser.so">
           <topicName>scan</topicName>
-          <frameName>base_link</frameName>
+          <frameName>laser</frameName>
         </plugin>
     </sensor>
   </gazebo>
-  <!--Send Position Information-->
   <gazebo>
     <plugin name="p3d_base_controller" filename="libgazebo_ros_p3d.so">
@@ -765,5 +858,5 @@
   	<bodyName>base_link</bodyName>
   	<topicName>base_pose_ground_truth</topicName>
-  	<gaussianNoise>0.01</gaussianNoise>
+  	<gaussianNoise>0</gaussianNoise>
   	<frameName>world</frameName>
   	<xyzOffsets>0 0 0</xyzOffsets>

Commit message: add rosbags

File: src/pkg/urdf/deepracer.xacro (robot description, xacro)
@@ -6,7 +6,4 @@
 <!-- Links and Joints -->
   <link name="base_link" />
-<gazebo reference="base_link">
-    <pose>0 0 0 0 0 0</pose>
-</gazebo>
   <link name="chassis">
     <inertial>
@@ -90,16 +87,4 @@
       velocity="100" />
   </joint>
-  <transmission name="left_rear_axle_trans">
-      <type>transmission_interface/SimpleTransmission</type>
-      <joint name="left_rear_wheel_joint">
-        <hardwareInterface>hardware_interface/EffortJointInterface</hardwareInterface>
-      </joint>
-      <actuator name="left_rear_axle_act">
-        <!-- This hardwareInterface element exists for compatibility
-             with ROS Hydro. -->
-        <hardwareInterface>hardware_interface/EffortJointInterface</hardwareInterface>
-        <mechanicalReduction>1</mechanicalReduction>
-      </actuator>
-  </transmission>
   <link
     name="right_rear_wheel">
@@ -153,16 +138,4 @@
       velocity="100" />
   </joint>
-    <transmission name="right_rear_axle_trans">
-      <type>transmission_interface/SimpleTransmission</type>
-      <joint name="right_rear_wheel_joint">
-        <hardwareInterface>hardware_interface/EffortJointInterface</hardwareInterface>
-      </joint>
-      <actuator name="right_rear_axle_act">
-        <!-- This hardwareInterface element exists for compatibility
-             with ROS Hydro. -->
-        <hardwareInterface>hardware_interface/EffortJointInterface</hardwareInterface>
-        <mechanicalReduction>1</mechanicalReduction>
-      </actuator>
-  </transmission>
   <link
     name="left_steering_hinge">
@@ -193,5 +166,5 @@
   <joint
     name="left_steering_hinge_joint"
-    type="continuous">
+    type="fixed">
     <origin
       xyz="0.082311 0.079601 0.011759"
@@ -209,16 +182,4 @@
       velocity="100" />
   </joint>
-  <transmission name="left_steering_trans">
-      <type>transmission_interface/SimpleTransmission</type>
-      <joint name="left_steering_hinge_joint">
-        <hardwareInterface>hardware_interface/EffortJointInterface</hardwareInterface>
-      </joint>
-      <actuator name="left_steering_act">
-        <!-- This hardwareInterface element exists for compatibility
-             with ROS Hydro. -->
-        <hardwareInterface>hardware_interface/EffortJointInterface</hardwareInterface>
-        <mechanicalReduction>1</mechanicalReduction>
-      </actuator>
-  </transmission>
   <link
     name="left_front_wheel">
@@ -272,16 +233,4 @@
       velocity="100" />
   </joint>
-  <transmission name="left_front_axle_trans">
-      <type>transmission_interface/SimpleTransmission</type>
-      <joint name="left_front_wheel_joint">
-        <hardwareInterface>hardware_interface/EffortJointInterface</hardwareInterface>
-      </joint>
-      <actuator name="left_front_axle_act">
-        <!-- This hardwareInterface element exists for compatibility
-             with ROS Hydro. -->
-        <hardwareInterface>hardware_interface/EffortJointInterface</hardwareInterface>
-        <mechanicalReduction>1</mechanicalReduction>
-      </actuator>
-  </transmission>
   <link
     name="right_steering_hinge">
@@ -312,5 +261,5 @@
   <joint
     name="right_steering_hinge_joint"
-    type="continuous">
+    type="fixed">
     <origin
       xyz="0.082311 -0.079601 0.011759"
@@ -328,16 +277,4 @@
       velocity="100" />
   </joint>
-  <transmission name="right_steering_trans">
-      <type>transmission_interface/SimpleTransmission</type>
-      <joint name="right_steering_hinge_joint">
-        <hardwareInterface>hardware_interface/EffortJointInterface</hardwareInterface>
-      </joint>
-      <actuator name="right_steering_act">
-        <!-- This hardwareInterface element exists for compatibility
-             with ROS Hydro. -->
-        <hardwareInterface>hardware_interface/EffortJointInterface</hardwareInterface>
-        <mechanicalReduction>1</mechanicalReduction>
-      </actuator>
-  </transmission>
   <link
     name="right_front_wheel">
@@ -391,16 +328,4 @@
       velocity="100" />
   </joint>
-    <transmission name="right_front_axle_trans">
-      <type>transmission_interface/SimpleTransmission</type>
-      <joint name="right_front_wheel_joint">
-        <hardwareInterface>hardware_interface/EffortJointInterface</hardwareInterface>
-      </joint>
-      <actuator name="right_front_axle_act">
-        <!-- This hardwareInterface element exists for compatibility
-             with ROS Hydro. -->
-        <hardwareInterface>hardware_interface/EffortJointInterface</hardwareInterface>
-        <mechanicalReduction>1</mechanicalReduction>
-      </actuator>
-  </transmission>
   <link
     name="zed_camera_link_leftcam">
@@ -536,5 +461,5 @@
         izz="1e-6" />
     </inertial>
-    <visual>
+<!--     <visual>
       <origin
         xyz="0 0 0"
@@ -544,5 +469,5 @@
           filename="package://pkg/meshes/deepracer/camera_link_rightcam.STL" />
       </geometry>
-    </visual>
+    </visual> -->
   </link>
   <joint
@@ -599,5 +524,5 @@
     <origin
       xyz="0.02913 0 0.16145"
-      rpy="0 0 0" />
+      rpy="0 0 3.1416" />
     <parent
       link="chassis" />
@@ -658,5 +583,4 @@
 <!-- Vehicle body -->
   <gazebo reference = "chassis">
-<pose>0 0 0 0 0 0</pose>
    <material>Gazebo/Grey</material>
    <mu1 value="0.0"/>
@@ -665,64 +589,55 @@
   </gazebo>
   <gazebo reference = "left_rear_wheel">
-<pose>0 0 0 0 0 0</pose>
    <material>Gazebo/DarkGrey</material>
-   <mu1 value="500"/>
-   <mu2 value="500"/>
+   <mu1 value="0.5"/>
+   <mu2 value="0.5"/>
    <kp  value="1000000.0" />
-   <kd  value="100000.0" />
+   <kd  value="1.0" />
    <fdir1 value="1 0 0"/>
   </gazebo>
   <gazebo reference = "left_front_wheel">
-<pose>0 0 0 0 0 0</pose>
    <material>Gazebo/DarkGrey</material>
-   <mu1 value="500"/>
-   <mu2 value="500"/>
+   <mu1 value="0.5"/>
+   <mu2 value="0.5"/>
    <kp  value="1000000.0" />
-   <kd  value="100000.0" />
+   <kd  value="1.0" />
    <fdir1 value="1 0 0"/>
   </gazebo>
   <gazebo reference = "right_rear_wheel">
-<pose>0 0 0 0 0 0</pose>
    <material>Gazebo/DarkGrey</material>
-   <mu1 value="500"/>
-   <mu2 value="500"/>
+   <mu1 value="0.5"/>
+   <mu2 value="0.5"/>
    <kp  value="1000000.0" />
-   <kd  value="100000.0" />
+   <kd  value="1.0" />
    <fdir1 value="1 0 0"/>
   </gazebo>
   <gazebo reference = "right_front_wheel">
-<pose>0 0 0 0 0 0</pose>
    <material>Gazebo/DarkGrey</material>
-   <mu1 value="500"/>
-   <mu2 value="500"/>
+   <mu1 value="0.5"/>
+   <mu2 value="0.5"/>
    <kp  value="1000000.0" />
-   <kd  value="100000.0" />
+   <kd  value="1.0" />
    <fdir1 value="1 0 0"/>
   </gazebo>
   <gazebo reference = "left_steering_hinge">
-<pose>0 0 0 0 0 0</pose>
    <material>Gazebo/DarkGrey</material>
   </gazebo>
   <gazebo reference = "right_steering_hinge">
-<pose>0 0 0 0 0 0</pose>
    <material>Gazebo/DarkGrey</material>
   </gazebo>
   <gazebo reference = "zed_camera_link_leftcam">
-<pose>0 0 0 0 0 0</pose>
    <material>Gazebo/DarkGrey</material>
   </gazebo>
   <gazebo reference = "zed_camera_link_rightcam">
-<pose>0 0 0 0 0 0</pose>
    <material>Gazebo/DarkGrey</material>
   </gazebo>
   <gazebo reference = "car_body_link_v3">
-<pose>0 0 0 0 0 0</pose>
    <material>Gazebo/Grey</material>
   </gazebo>
 <!-- Chassis Controller-->
-   <!--gazebo>
+   <gazebo>
     <plugin name="skid_steer_drive_controller" filename="libgazebo_ros_skid_steer_drive.so">
       <updateRate>30</updateRate>
-      <robotNamespace>/</robotNamespace>
+      <robotNamespace>$(arg bodyframe)</robotNamespace>
       <leftFrontJoint>left_front_wheel_joint</leftFrontJoint>
       <rightFrontJoint>right_front_wheel_joint</rightFrontJoint>
@@ -731,20 +646,13 @@
       <wheelSeparation>0.159202</wheelSeparation>
       <wheelDiameter>0.06</wheelDiameter>
-      <robotBaseFrame>base_link</robotBaseFrame>
+      <robotBaseFrame>$(arg bodyframe)/base_link</robotBaseFrame>
       <torque>20</torque>
       <commandTopic>cmd_vel</commandTopic>
       <odometryTopic>odom</odometryTopic>
       <odometryFrame>odom</odometryFrame>
-      <covariance_x>0</covariance_x>
-      <covariance_y>0</covariance_y>
-      <covariance_yaw>0</covariance_yaw>
+      <covariance_x>0.0001</covariance_x>
+      <covariance_y>0.0001</covariance_y>
+      <covariance_yaw>0.0001</covariance_yaw>
       <broadcastTF>true</broadcastTF>
-    </plugin>
-  </gazebo-->
-  <gazebo>
-    <plugin name="gazebo_ros_control" filename="libgazebo_ros_control.so">
-    <legacyModeNS>true</legacyModeNS>
-    <robotSimType>gazebo_ros_control/DefaultRobotHWSim</robotSimType>
-    <robotNamespace>$(arg bodyframe)</robotNamespace>
     </plugin>
   </gazebo>
@@ -824,5 +732,5 @@
       <pose>0 0 0 0 0 0</pose>
       <visualize>false</visualize>
-      <update_rate>10</update_rate>
+      <update_rate>30</update_rate>
       <ray>
         <scan>
@@ -830,8 +738,6 @@
             <samples>600</samples>
             <resolution>1</resolution>
-             <min_angle>-3.1415926</min_angle>
-             <max_angle>3.1415926</max_angle>
-            <!--min_angle>0.52351</min_angle>
-            <max_angle>5.75949</max_angle-->
+            <min_angle>-2.61799</min_angle>
+            <max_angle>2.61799</max_angle>
           </horizontal>
         </scan>
@@ -843,13 +749,14 @@
         <noise>
           <mean>0.0</mean>
-          <stddev>0</stddev>
+          <stddev>0.01</stddev>
         </noise>
       </ray>
        <plugin name="rp_lidar" filename="libgazebo_ros_laser.so">
           <topicName>scan</topicName>
-          <frameName>laser</frameName>
+          <frameName>base_link</frameName>
         </plugin>
     </sensor>
   </gazebo>
+  <!--Send Position Information-->
   <gazebo>
     <plugin name="p3d_base_controller" filename="libgazebo_ros_p3d.so">
@@ -858,5 +765,5 @@
   	<bodyName>base_link</bodyName>
   	<topicName>base_pose_ground_truth</topicName>
-  	<gaussianNoise>0</gaussianNoise>
+  	<gaussianNoise>0.01</gaussianNoise>
   	<frameName>world</frameName>
   	<xyzOffsets>0 0 0</xyzOffsets>
