Commit message: fixed

File: src/site_model/urdf/site_model.urdf.xacro (robot description, xacro)
@@ -2314,3 +2314,817 @@
     <xacro:deepracer parent="base_link" name="deepracer">
   </xacro:deepracer>-->
+  <!-- <link name="chassis">
+    <inertial>
+      <origin
+        xyz="0 0 0"
+        rpy="0 0 0" />
+      <mass
+        value="5.0" />
+      <inertia
+        ixx="0.010609"
+        ixy="0"
+        ixz="0"
+        iyy="0.050409"
+        iyz="0"
+        izz="0.05865" />
+    </inertial>
+    <visual>
+      <origin
+        xyz="0 0 0"
+        rpy="0 0 0" />
+      <geometry>
+        <mesh
+          filename="package://pkg/meshes/deepracer/chassis.STL" />
+      </geometry>
+    </visual>
+  </link>
+  <joint name="base_link_joint" type="fixed">
+    <origin xyz="0 0 0.023249" rpy="0 0 0" />
+    <parent link="base_link" />
+    <child link="chassis" />
+  </joint>
+  <link
+    name="left_rear_wheel">
+    <inertial>
+      <origin
+        xyz="0 0 0"
+        rpy="0 0 0" />
+      <mass
+        value="0.34055" />
+      <inertia
+        ixx="0.00026046"
+        ixy="0"
+        ixz="0"
+        iyy="0.00041226"
+        iyz="0"
+        izz="0.00026046" />
+    </inertial>
+    <visual>
+      <origin
+        xyz="0 0 0"
+        rpy="0 0 0" />
+      <geometry>
+        <mesh
+          filename="package://pkg/meshes/deepracer/left_rear_wheel.STL" />
+      </geometry>
+    </visual>
+    <collision>
+      <origin
+        xyz="0 0 0"
+        rpy="0 0 0" />
+      <geometry>
+        <mesh
+          filename="package://pkg/meshes/deepracer/left_rear_wheel.STL" />
+      </geometry>
+    </collision>
+  </link>
+  <joint
+    name="left_rear_wheel_joint"
+    type="continuous">
+    <origin
+      xyz="-0.081663 0.08105 0.01575"
+      rpy="0 0 0" />
+    <parent
+      link="chassis" />
+    <child
+      link="left_rear_wheel" />
+    <axis
+      xyz="0 1 0" />
+    <limit
+      effort="10"
+      velocity="100" />
+  </joint>
+  <transmission name="left_rear_axle_trans">
+      <type>transmission_interface/SimpleTransmission</type>
+      <joint name="left_rear_wheel_joint">
+        <hardwareInterface>hardware_interface/EffortJointInterface</hardwareInterface>
+      </joint>
+      <actuator name="left_rear_axle_act">
+        <!-- This hardwareInterface element exists for compatibility
+             with ROS Hydro. -->
+        <hardwareInterface>hardware_interface/EffortJointInterface</hardwareInterface>
+        <mechanicalReduction>1</mechanicalReduction>
+      </actuator>
+  </transmission>
+  <link
+    name="right_rear_wheel">
+    <inertial>
+      <origin
+        xyz="0 0 0"
+        rpy="0 0 0" />
+      <mass
+        value="0.34055" />
+      <inertia
+        ixx="0.00026046"
+        ixy="0"
+        ixz="0"
+        iyy="0.00041226"
+        iyz="0"
+        izz="0.00026046" />
+    </inertial>
+    <visual>
+      <origin
+        xyz="0 0 0"
+        rpy="0 0 0" />
+      <geometry>
+        <mesh
+          filename="package://pkg/meshes/deepracer/right_rear_wheel.STL" />
+      </geometry>
+    </visual>
+    <collision>
+      <origin
+        xyz="0 0 0"
+        rpy="0 0 0" />
+      <geometry>
+        <mesh
+          filename="package://pkg/meshes/deepracer/right_rear_wheel.STL" />
+      </geometry>
+    </collision>
+  </link>
+  <joint
+    name="right_rear_wheel_joint"
+    type="continuous">
+    <origin
+      xyz="-0.081663 -0.08105 0.01575"
+      rpy="0 0 0" />
+    <parent
+      link="chassis" />
+    <child
+      link="right_rear_wheel" />
+    <axis
+      xyz="0 1 0" />
+    <limit
+      effort="10"
+      velocity="100" />
+  </joint>
+    <transmission name="right_rear_axle_trans">
+      <type>transmission_interface/SimpleTransmission</type>
+      <joint name="right_rear_wheel_joint">
+        <hardwareInterface>hardware_interface/EffortJointInterface</hardwareInterface>
+      </joint>
+      <actuator name="right_rear_axle_act">
+        <!-- This hardwareInterface element exists for compatibility
+             with ROS Hydro. -->
+        <hardwareInterface>hardware_interface/EffortJointInterface</hardwareInterface>
+        <mechanicalReduction>1</mechanicalReduction>
+      </actuator>
+  </transmission>
+  <link
+    name="left_steering_hinge">
+    <inertial>
+      <origin
+        xyz="0 0 0"
+        rpy="0 0 0" />
+      <mass
+        value="0.1" />
+      <inertia
+        ixx="4E-06"
+        ixy="0"
+        ixz="0"
+        iyy="4E-06"
+        iyz="0"
+        izz="4E-06" />
+      </inertial>
+    <visual>
+      <origin
+        xyz="0 0 0"
+        rpy="0 0 0" />
+      <geometry>
+        <mesh
+          filename="package://pkg/meshes/deepracer/left_steering_hinge.STL" />
+      </geometry>
+    </visual>
+  </link>
+  <joint
+    name="left_steering_hinge_joint"
+    type="continuous">
+    <origin
+      xyz="0.082311 0.079601 0.011759"
+      rpy="0 0 0" />
+    <parent
+      link="chassis" />
+    <child
+      link="left_steering_hinge" />
+    <axis
+      xyz="0 0 1" />
+    <limit
+      lower="-1"
+      upper="1"
+      effort="10"
+      velocity="100" />
+  </joint>
+  <transmission name="left_steering_trans">
+      <type>transmission_interface/SimpleTransmission</type>
+      <joint name="left_steering_hinge_joint">
+        <hardwareInterface>hardware_interface/EffortJointInterface</hardwareInterface>
+      </joint>
+      <actuator name="left_steering_act">
+        <!-- This hardwareInterface element exists for compatibility
+             with ROS Hydro. -->
+        <hardwareInterface>hardware_interface/EffortJointInterface</hardwareInterface>
+        <mechanicalReduction>1</mechanicalReduction>
+      </actuator>
+  </transmission>
+  <link
+    name="left_front_wheel">
+    <inertial>
+      <origin
+        xyz="0 0 0"
+        rpy="0 0 0" />
+      <mass
+        value="0.34055" />
+      <inertia
+        ixx="0.00026046"
+        ixy="0"
+        ixz="0"
+        iyy="0.00041226"
+        iyz="0"
+        izz="0.00026046" />
+    </inertial>
+    <visual>
+      <origin
+        xyz="0 0 0"
+        rpy="0 0 0" />
+      <geometry>
+        <mesh
+          filename="package://pkg/meshes/deepracer/left_front_wheel.STL" />
+      </geometry>
+    </visual>
+    <collision>
+      <origin
+        xyz="0 0 0"
+        rpy="0 0 0" />
+      <geometry>
+        <mesh
+          filename="package://pkg/meshes/deepracer/left_front_wheel.STL" />
+      </geometry>
+    </collision>
+  </link>
+  <joint
+    name="left_front_wheel_joint"
+    type="continuous">
+    <origin
+      xyz="0 0 0"
+      rpy="0 0 0" />
+    <parent
+      link="left_steering_hinge" />
+    <child
+      link="left_front_wheel" />
+    <axis
+      xyz="0 1 0" />
+    <limit
+      effort="10"
+      velocity="100" />
+  </joint>
+  <transmission name="left_front_axle_trans">
+      <type>transmission_interface/SimpleTransmission</type>
+      <joint name="left_front_wheel_joint">
+        <hardwareInterface>hardware_interface/EffortJointInterface</hardwareInterface>
+      </joint>
+      <actuator name="left_front_axle_act">
+        <!-- This hardwareInterface element exists for compatibility
+             with ROS Hydro. -->
+        <hardwareInterface>hardware_interface/EffortJointInterface</hardwareInterface>
+        <mechanicalReduction>1</mechanicalReduction>
+      </actuator>
+  </transmission>
+  <link
+    name="right_steering_hinge">
+    <inertial>
+      <origin
+        xyz="0 0 0"
+        rpy="0 0 0" />
+      <mass
+        value="0.1" />
+      <inertia
+        ixx="4E-06"
+        ixy="0"
+        ixz="0"
+        iyy="4E-06"
+        iyz="0"
+        izz="4E-06" />
+    </inertial>
+    <visual>
+      <origin
+        xyz="0 0 0"
+        rpy="0 0 0" />
+      <geometry>
+        <mesh
+          filename="package://pkg/meshes/deepracer/right_steering_hinge.STL" />
+      </geometry>
+    </visual>
+  </link>
+  <joint
+    name="right_steering_hinge_joint"
+    type="continuous">
+    <origin
+      xyz="0.082311 -0.079601 0.011759"
+      rpy="0 0 0" />
+    <parent
+      link="chassis" />
+    <child
+      link="right_steering_hinge" />
+    <axis
+      xyz="0 0 1" />
+    <limit
+      lower="-1"
+      upper="1"
+      effort="10"
+      velocity="100" />
+  </joint>
+  <transmission name="right_steering_trans">
+      <type>transmission_interface/SimpleTransmission</type>
+      <joint name="right_steering_hinge_joint">
+        <hardwareInterface>hardware_interface/EffortJointInterface</hardwareInterface>
+      </joint>
+      <actuator name="right_steering_act">
+        <!-- This hardwareInterface element exists for compatibility
+             with ROS Hydro. -->
+        <hardwareInterface>hardware_interface/EffortJointInterface</hardwareInterface>
+        <mechanicalReduction>1</mechanicalReduction>
+      </actuator>
+  </transmission>
+  <link
+    name="right_front_wheel">
+    <inertial>
+      <origin
+        xyz="0 0 0"
+        rpy="0 0 0" />
+      <mass
+        value="0.34055" />
+      <inertia
+        ixx="0.00026046"
+        ixy="0"
+        ixz="0"
+        iyy="0.00041226"
+        iyz="0"
+        izz="0.00026046" />
+    </inertial>
+    <visual>
+      <origin
+        xyz="0 0 0"
+        rpy="0 0 0" />
+      <geometry>
+        <mesh
+          filename="package://pkg/meshes/deepracer/right_front_wheel.STL" />
+      </geometry>
+    </visual>
+    <collision>
+      <origin
+        xyz="0 0 0"
+        rpy="0 0 0" />
+      <geometry>
+        <mesh
+          filename="package://pkg/meshes/deepracer/right_front_wheel.STL" />
+      </geometry>
+    </collision>
+  </link>
+  <joint
+    name="right_front_wheel_joint"
+    type="continuous">
+    <origin
+      xyz="0 0 0"
+      rpy="0 0 0" />
+    <parent
+      link="right_steering_hinge" />
+    <child
+      link="right_front_wheel" />
+    <axis
+      xyz="0 1 0" />
+    <limit
+      effort="10"
+      velocity="100" />
+  </joint>
+    <transmission name="right_front_axle_trans">
+      <type>transmission_interface/SimpleTransmission</type>
+      <joint name="right_front_wheel_joint">
+        <hardwareInterface>hardware_interface/EffortJointInterface</hardwareInterface>
+      </joint>
+      <actuator name="right_front_axle_act">
+        <!-- This hardwareInterface element exists for compatibility
+             with ROS Hydro. -->
+        <hardwareInterface>hardware_interface/EffortJointInterface</hardwareInterface>
+        <mechanicalReduction>1</mechanicalReduction>
+      </actuator>
+  </transmission>
+  <link
+    name="zed_camera_link_leftcam">
+    <inertial>
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
Commit message: fixed

File: src/site_model/urdf/site_model.urdf.xacro (robot description, xacro)
@@ -2314,817 +2314,3 @@
     <xacro:deepracer parent="base_link" name="deepracer">
   </xacro:deepracer>-->
-  <!-- <link name="chassis">
-    <inertial>
-      <origin
-        xyz="0 0 0"
-        rpy="0 0 0" />
-      <mass
-        value="5.0" />
-      <inertia
-        ixx="0.010609"
-        ixy="0"
-        ixz="0"
-        iyy="0.050409"
-        iyz="0"
-        izz="0.05865" />
-    </inertial>
-    <visual>
-      <origin
-        xyz="0 0 0"
-        rpy="0 0 0" />
-      <geometry>
-        <mesh
-          filename="package://pkg/meshes/deepracer/chassis.STL" />
-      </geometry>
-    </visual>
-  </link>
-  <joint name="base_link_joint" type="fixed">
-    <origin xyz="0 0 0.023249" rpy="0 0 0" />
-    <parent link="base_link" />
-    <child link="chassis" />
-  </joint>
-  <link
-    name="left_rear_wheel">
-    <inertial>
-      <origin
-        xyz="0 0 0"
-        rpy="0 0 0" />
-      <mass
-        value="0.34055" />
-      <inertia
-        ixx="0.00026046"
-        ixy="0"
-        ixz="0"
-        iyy="0.00041226"
-        iyz="0"
-        izz="0.00026046" />
-    </inertial>
-    <visual>
-      <origin
-        xyz="0 0 0"
-        rpy="0 0 0" />
-      <geometry>
-        <mesh
-          filename="package://pkg/meshes/deepracer/left_rear_wheel.STL" />
-      </geometry>
-    </visual>
-    <collision>
-      <origin
-        xyz="0 0 0"
-        rpy="0 0 0" />
-      <geometry>
-        <mesh
-          filename="package://pkg/meshes/deepracer/left_rear_wheel.STL" />
-      </geometry>
-    </collision>
-  </link>
-  <joint
-    name="left_rear_wheel_joint"
-    type="continuous">
-    <origin
-      xyz="-0.081663 0.08105 0.01575"
-      rpy="0 0 0" />
-    <parent
-      link="chassis" />
-    <child
-      link="left_rear_wheel" />
-    <axis
-      xyz="0 1 0" />
-    <limit
-      effort="10"
-      velocity="100" />
-  </joint>
-  <transmission name="left_rear_axle_trans">
-      <type>transmission_interface/SimpleTransmission</type>
-      <joint name="left_rear_wheel_joint">
-        <hardwareInterface>hardware_interface/EffortJointInterface</hardwareInterface>
-      </joint>
-      <actuator name="left_rear_axle_act">
-        <!-- This hardwareInterface element exists for compatibility
-             with ROS Hydro. -->
-        <hardwareInterface>hardware_interface/EffortJointInterface</hardwareInterface>
-        <mechanicalReduction>1</mechanicalReduction>
-      </actuator>
-  </transmission>
-  <link
-    name="right_rear_wheel">
-    <inertial>
-      <origin
-        xyz="0 0 0"
-        rpy="0 0 0" />
-      <mass
-        value="0.34055" />
-      <inertia
-        ixx="0.00026046"
-        ixy="0"
-        ixz="0"
-        iyy="0.00041226"
-        iyz="0"
-        izz="0.00026046" />
-    </inertial>
-    <visual>
-      <origin
-        xyz="0 0 0"
-        rpy="0 0 0" />
-      <geometry>
-        <mesh
-          filename="package://pkg/meshes/deepracer/right_rear_wheel.STL" />
-      </geometry>
-    </visual>
-    <collision>
-      <origin
-        xyz="0 0 0"
-        rpy="0 0 0" />
-      <geometry>
-        <mesh
-          filename="package://pkg/meshes/deepracer/right_rear_wheel.STL" />
-      </geometry>
-    </collision>
-  </link>
-  <joint
-    name="right_rear_wheel_joint"
-    type="continuous">
-    <origin
-      xyz="-0.081663 -0.08105 0.01575"
-      rpy="0 0 0" />
-    <parent
-      link="chassis" />
-    <child
-      link="right_rear_wheel" />
-    <axis
-      xyz="0 1 0" />
-    <limit
-      effort="10"
-      velocity="100" />
-  </joint>
-    <transmission name="right_rear_axle_trans">
-      <type>transmission_interface/SimpleTransmission</type>
-      <joint name="right_rear_wheel_joint">
-        <hardwareInterface>hardware_interface/EffortJointInterface</hardwareInterface>
-      </joint>
-      <actuator name="right_rear_axle_act">
-        <!-- This hardwareInterface element exists for compatibility
-             with ROS Hydro. -->
-        <hardwareInterface>hardware_interface/EffortJointInterface</hardwareInterface>
-        <mechanicalReduction>1</mechanicalReduction>
-      </actuator>
-  </transmission>
-  <link
-    name="left_steering_hinge">
-    <inertial>
-      <origin
-        xyz="0 0 0"
-        rpy="0 0 0" />
-      <mass
-        value="0.1" />
-      <inertia
-        ixx="4E-06"
-        ixy="0"
-        ixz="0"
-        iyy="4E-06"
-        iyz="0"
-        izz="4E-06" />
-      </inertial>
-    <visual>
-      <origin
-        xyz="0 0 0"
-        rpy="0 0 0" />
-      <geometry>
-        <mesh
-          filename="package://pkg/meshes/deepracer/left_steering_hinge.STL" />
-      </geometry>
-    </visual>
-  </link>
-  <joint
-    name="left_steering_hinge_joint"
-    type="continuous">
-    <origin
-      xyz="0.082311 0.079601 0.011759"
-      rpy="0 0 0" />
-    <parent
-      link="chassis" />
-    <child
-      link="left_steering_hinge" />
-    <axis
-      xyz="0 0 1" />
-    <limit
-      lower="-1"
-      upper="1"
-      effort="10"
-      velocity="100" />
-  </joint>
-  <transmission name="left_steering_trans">
-      <type>transmission_interface/SimpleTransmission</type>
-      <joint name="left_steering_hinge_joint">
-        <hardwareInterface>hardware_interface/EffortJointInterface</hardwareInterface>
-      </joint>
-      <actuator name="left_steering_act">
-        <!-- This hardwareInterface element exists for compatibility
-             with ROS Hydro. -->
-        <hardwareInterface>hardware_interface/EffortJointInterface</hardwareInterface>
-        <mechanicalReduction>1</mechanicalReduction>
-      </actuator>
-  </transmission>
-  <link
-    name="left_front_wheel">
-    <inertial>
-      <origin
-        xyz="0 0 0"
-        rpy="0 0 0" />
-      <mass
-        value="0.34055" />
-      <inertia
-        ixx="0.00026046"
-        ixy="0"
-        ixz="0"
-        iyy="0.00041226"
-        iyz="0"
-        izz="0.00026046" />
-    </inertial>
-    <visual>
-      <origin
-        xyz="0 0 0"
-        rpy="0 0 0" />
-      <geometry>
-        <mesh
-          filename="package://pkg/meshes/deepracer/left_front_wheel.STL" />
-      </geometry>
-    </visual>
-    <collision>
-      <origin
-        xyz="0 0 0"
-        rpy="0 0 0" />
-      <geometry>
-        <mesh
-          filename="package://pkg/meshes/deepracer/left_front_wheel.STL" />
-      </geometry>
-    </collision>
-  </link>
-  <joint
-    name="left_front_wheel_joint"
-    type="continuous">
-    <origin
-      xyz="0 0 0"
-      rpy="0 0 0" />
-    <parent
-      link="left_steering_hinge" />
-    <child
-      link="left_front_wheel" />
-    <axis
-      xyz="0 1 0" />
-    <limit
-      effort="10"
-      velocity="100" />
-  </joint>
-  <transmission name="left_front_axle_trans">
-      <type>transmission_interface/SimpleTransmission</type>
-      <joint name="left_front_wheel_joint">
-        <hardwareInterface>hardware_interface/EffortJointInterface</hardwareInterface>
-      </joint>
-      <actuator name="left_front_axle_act">
-        <!-- This hardwareInterface element exists for compatibility
-             with ROS Hydro. -->
-        <hardwareInterface>hardware_interface/EffortJointInterface</hardwareInterface>
-        <mechanicalReduction>1</mechanicalReduction>
-      </actuator>
-  </transmission>
-  <link
-    name="right_steering_hinge">
-    <inertial>
-      <origin
-        xyz="0 0 0"
-        rpy="0 0 0" />
-      <mass
-        value="0.1" />
-      <inertia
-        ixx="4E-06"
-        ixy="0"
-        ixz="0"
-        iyy="4E-06"
-        iyz="0"
-        izz="4E-06" />
-    </inertial>
-    <visual>
-      <origin
-        xyz="0 0 0"
-        rpy="0 0 0" />
-      <geometry>
-        <mesh
-          filename="package://pkg/meshes/deepracer/right_steering_hinge.STL" />
-      </geometry>
-    </visual>
-  </link>
-  <joint
-    name="right_steering_hinge_joint"
-    type="continuous">
-    <origin
-      xyz="0.082311 -0.079601 0.011759"
-      rpy="0 0 0" />
-    <parent
-      link="chassis" />
-    <child
-      link="right_steering_hinge" />
-    <axis
-      xyz="0 0 1" />
-    <limit
-      lower="-1"
-      upper="1"
-      effort="10"
-      velocity="100" />
-  </joint>
-  <transmission name="right_steering_trans">
-      <type>transmission_interface/SimpleTransmission</type>
-      <joint name="right_steering_hinge_joint">
-        <hardwareInterface>hardware_interface/EffortJointInterface</hardwareInterface>
-      </joint>
-      <actuator name="right_steering_act">
-        <!-- This hardwareInterface element exists for compatibility
-             with ROS Hydro. -->
-        <hardwareInterface>hardware_interface/EffortJointInterface</hardwareInterface>
-        <mechanicalReduction>1</mechanicalReduction>
-      </actuator>
-  </transmission>
-  <link
-    name="right_front_wheel">
-    <inertial>
-      <origin
-        xyz="0 0 0"
-        rpy="0 0 0" />
-      <mass
-        value="0.34055" />
-      <inertia
-        ixx="0.00026046"
-        ixy="0"
-        ixz="0"
-        iyy="0.00041226"
-        iyz="0"
-        izz="0.00026046" />
-    </inertial>
-    <visual>
-      <origin
-        xyz="0 0 0"
-        rpy="0 0 0" />
-      <geometry>
-        <mesh
-          filename="package://pkg/meshes/deepracer/right_front_wheel.STL" />
-      </geometry>
-    </visual>
-    <collision>
-      <origin
-        xyz="0 0 0"
-        rpy="0 0 0" />
-      <geometry>
-        <mesh
-          filename="package://pkg/meshes/deepracer/right_front_wheel.STL" />
-      </geometry>
-    </collision>
-  </link>
-  <joint
-    name="right_front_wheel_joint"
-    type="continuous">
-    <origin
-      xyz="0 0 0"
-      rpy="0 0 0" />
-    <parent
-      link="right_steering_hinge" />
-    <child
-      link="right_front_wheel" />
-    <axis
-      xyz="0 1 0" />
-    <limit
-      effort="10"
-      velocity="100" />
-  </joint>
-    <transmission name="right_front_axle_trans">
-      <type>transmission_interface/SimpleTransmission</type>
-      <joint name="right_front_wheel_joint">
-        <hardwareInterface>hardware_interface/EffortJointInterface</hardwareInterface>
-      </joint>
-      <actuator name="right_front_axle_act">
-        <!-- This hardwareInterface element exists for compatibility
-             with ROS Hydro. -->
-        <hardwareInterface>hardware_interface/EffortJointInterface</hardwareInterface>
-        <mechanicalReduction>1</mechanicalReduction>
-      </actuator>
-  </transmission>
-  <link
-    name="zed_camera_link_leftcam">
-    <inertial>
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