Commit message: add twe new cameras && modify speed of car

File: src/site_model/urdf/site_model.urdf.xacro (robot description, xacro)
@@ -99,4 +99,12 @@
   </gazebo>
   <gazebo reference="camera44_Link">
+    <material>Gazebo/Black</material>
+    <turnGravityOff>false</turnGravityOff>
+  </gazebo>
+  <gazebo reference="camera5_Link">
+    <material>Gazebo/Black</material>
+    <turnGravityOff>false</turnGravityOff>
+  </gazebo>
+  <gazebo reference="camera6_Link">
     <material>Gazebo/Black</material>
     <turnGravityOff>false</turnGravityOff>
@@ -1257,4 +1265,186 @@
     </sensor>
   </gazebo>
+  <!-- camera5 -->
+  <link
+    name="camera5_Link">
+    <inertial>
+      <origin
+        xyz="0.000108384331294675 -0.00200274517214477 0.0112406574811803"
+        rpy="0 0 0" />
+      <mass
+        value="0.814135587689854" />
+      <inertia
+        ixx="0.000299485503699371"
+        ixy="-8.50166027613617E-08"
+        ixz="-2.30003016200203E-09"
+        iyy="0.000280071339845325"
+        iyz="2.45106701788653E-06"
+        izz="0.000373933133462947" />
+    </inertial>
+    <visual>
+      <origin
+        xyz="-0.02 0 0"
+        rpy="0 0 0" />
+      <geometry>
+        <mesh
+          filename="package://site_model/meshes/camera5_Link.STL" />
+      </geometry>
+      <material
+        name="">
+        <color
+          rgba="0.529411764705882 0.549019607843137 0.549019607843137 1" />
+      </material>
+    </visual>
+    <collision>
+      <origin
+        xyz="0 0 0"
+        rpy="0 0 0" />
+      <geometry>
+        <mesh
+          filename="package://site_model/meshes/camera5_Link.STL" />
+      </geometry>
+    </collision>
+  </link>
+  <joint
+    name="camera5"
+    type="fixed">
+    <origin
+      xyz="-1.4 2 0.8"
+      rpy="0 0 0.792156862745098" />
+    <parent
+      link="base_link" />
+    <child
+      link="camera5_Link" />
+    <axis
+      xyz="0 0 0" />
+  </joint>
+<gazebo reference="camera5_Link">
+    <sensor type="camera" name="camera5">
+      <pose>0 0 0 0 0 0</pose>
+      <update_rate>15.0</update_rate>
+      <camera name="camera5">
+        <horizontal_fov>1.13</horizontal_fov>
+        <image>
+          <width>640</width>
+          <height>480</height>
+          <format>R8G8B8</format>
+        </image>
+        <clip>
+          <near>0.02</near>
+          <far>300</far>
+        </clip>
+        <noise>
+          <type>gaussian</type>
+          <mean>0.0</mean>
+          <stddev>0.007</stddev>
+        </noise>
+      </camera>
+      <plugin name="camera_controller" filename="libgazebo_ros_camera.so">
+        <alwaysOn>true</alwaysOn>
+        <updateRate>60</updateRate>
+        <cameraName>camera5</cameraName>
+        <imageTopicName>/image_raw_5</imageTopicName>
+        <cameraInfoTopicName>camera_info</cameraInfoTopicName>
+        <frameName>camera5_Link</frameName>
+        <hackBaseline>0.0</hackBaseline>
+        <distortionK1>0.0</distortionK1>
+        <distortionK2>0.0</distortionK2>
+        <distortionK3>0.0</distortionK3>
+        <distortionT1>0.0</distortionT1>
+        <distortionT2>0.0</distortionT2>
+      </plugin>
+    </sensor>
+  </gazebo>
+  <!-- camera6 -->
+  <link
+    name="camera6_Link">
+    <inertial>
+      <origin
+        xyz="0.000108384331294675 -0.00200274517214477 0.0112406574811803"
+        rpy="0 0 0" />
+      <mass
+        value="0.814135587689854" />
+      <inertia
+        ixx="0.000299485503699371"
+        ixy="-8.50166027613617E-08"
+        ixz="-2.30003016200203E-09"
+        iyy="0.000280071339845325"
+        iyz="2.45106701788653E-06"
+        izz="0.000373933133462947" />
+    </inertial>
+    <visual>
+      <origin
+        xyz="-0.02 0 0"
+        rpy="0 0 0" />
+      <geometry>
+        <mesh
+          filename="package://site_model/meshes/camera6_Link.STL" />
+      </geometry>
+      <material
+        name="">
+        <color
+          rgba="0.529411764705882 0.549019607843137 0.549019607843137 1" />
+      </material>
+    </visual>
+    <collision>
+      <origin
+        xyz="0 0 0"
+        rpy="0 0 0" />
+      <geometry>
+        <mesh
+          filename="package://site_model/meshes/camera6_Link.STL" />
+      </geometry>
+    </collision>
+  </link>
+  <joint
+    name="camera6"
+    type="fixed">
+    <origin
+      xyz="1 2 0.8"
+      rpy="0 0 2.356194490192345" />
+    <parent
+      link="base_link" />
+    <child
+      link="camera6_Link" />
+    <axis
+      xyz="0 0 0" />
+  </joint>
+<gazebo reference="camera6_Link">
+    <sensor type="camera" name="camera6">
+      <pose>0 0 0 0 0 0</pose>
+      <update_rate>15.0</update_rate>
+      <camera name="camera6">
+        <horizontal_fov>1.13</horizontal_fov>
+        <image>
+          <width>640</width>
+          <height>480</height>
+          <format>R8G8B8</format>
+        </image>
+        <clip>
+          <near>0.02</near>
+          <far>300</far>
+        </clip>
+        <noise>
+          <type>gaussian</type>
+          <mean>0.0</mean>
+          <stddev>0.007</stddev>
+        </noise>
+      </camera>
+      <plugin name="camera_controller" filename="libgazebo_ros_camera.so">
+        <alwaysOn>true</alwaysOn>
+        <updateRate>60</updateRate>
+        <cameraName>camera6</cameraName>
+        <imageTopicName>/image_raw_6</imageTopicName>
+        <cameraInfoTopicName>camera_info</cameraInfoTopicName>
+        <frameName>camera6_Link</frameName>
+        <hackBaseline>0.0</hackBaseline>
+        <distortionK1>0.0</distortionK1>
+        <distortionK2>0.0</distortionK2>
+        <distortionK3>0.0</distortionK3>
+        <distortionT1>0.0</distortionT1>
+        <distortionT2>0.0</distortionT2>
+      </plugin>
+    </sensor>
+  </gazebo>
   <!-- Lidar_2 points3 -->
   <joint name="velodyne2_base_mount_joint" type="fixed">

Commit message: add camera7

File: src/site_model/urdf/site_model.urdf.xacro (robot description, xacro)
@@ -107,4 +107,20 @@
   </gazebo>
   <gazebo reference="camera6_Link">
+    <material>Gazebo/Black</material>
+    <turnGravityOff>false</turnGravityOff>
+  </gazebo>
+  <gazebo reference="camera7_Link">
+    <material>Gazebo/Black</material>
+    <turnGravityOff>false</turnGravityOff>
+  </gazebo>
+  <gazebo reference="camera8_Link">
+    <material>Gazebo/Black</material>
+    <turnGravityOff>false</turnGravityOff>
+  </gazebo>
+  <gazebo reference="camera9_Link">
+    <material>Gazebo/Black</material>
+    <turnGravityOff>false</turnGravityOff>
+  </gazebo>
+  <gazebo reference="camera10_Link">
     <material>Gazebo/Black</material>
     <turnGravityOff>false</turnGravityOff>
@@ -1310,5 +1326,5 @@
     type="fixed">
     <origin
-      xyz="-1.4 2 0.8"
+      xyz="-1.4 2 0.7"
       rpy="0 0 0.792156862745098" />
     <parent
@@ -1401,5 +1417,5 @@
     type="fixed">
     <origin
-      xyz="1 2 0.8"
+      xyz="1.1 1.9 0.7"
       rpy="0 0 2.356194490192345" />
     <parent
@@ -1438,4 +1454,95 @@
         <cameraInfoTopicName>camera_info</cameraInfoTopicName>
         <frameName>camera6_Link</frameName>
+        <hackBaseline>0.0</hackBaseline>
+        <distortionK1>0.0</distortionK1>
+        <distortionK2>0.0</distortionK2>
+        <distortionK3>0.0</distortionK3>
+        <distortionT1>0.0</distortionT1>
+        <distortionT2>0.0</distortionT2>
+      </plugin>
+    </sensor>
+  </gazebo>
+  <!-- camera7 -->
+  <link
+    name="camera7_Link">
+    <inertial>
+      <origin
+        xyz="0.000108384331294675 -0.00200274517214477 0.0112406574811803"
+        rpy="0 0 0" />
+      <mass
+        value="0.814135587689854" />
+      <inertia
+        ixx="0.000299485503699371"
+        ixy="-8.50166027613617E-08"
+        ixz="-2.30003016200203E-09"
+        iyy="0.000280071339845325"
+        iyz="2.45106701788653E-06"
+        izz="0.000373933133462947" />
+    </inertial>
+    <visual>
+      <origin
+        xyz="-0.02 0 0"
+        rpy="0 0 0" />
+      <geometry>
+        <mesh
+          filename="package://site_model/meshes/camera7_Link.STL" />
+      </geometry>
+      <material
+        name="">
+        <color
+          rgba="0.529411764705882 0.549019607843137 0.549019607843137 1" />
+      </material>
+    </visual>
+    <collision>
+      <origin
+        xyz="0 0 0"
+        rpy="0 0 0" />
+      <geometry>
+        <mesh
+          filename="package://site_model/meshes/camera7_Link.STL" />
+      </geometry>
+    </collision>
+  </link>
+  <joint
+    name="camera7"
+    type="fixed">
+    <origin
+      xyz="-0.75 2.7 0.7"
+      rpy="0 0 0.3490658503988659" />
+    <parent
+      link="base_link" />
+    <child
+      link="camera7_Link" />
+    <axis
+      xyz="0 0 0" />
+  </joint>
+<gazebo reference="camera7_Link">
+    <sensor type="camera" name="camera7">
+      <pose>0 0 0 0 0 0</pose>
+      <update_rate>15.0</update_rate>
+      <camera name="camera7">
+        <horizontal_fov>1.13</horizontal_fov>
+        <image>
+          <width>640</width>
+          <height>480</height>
+          <format>R8G8B8</format>
+        </image>
+        <clip>
+          <near>0.02</near>
+          <far>300</far>
+        </clip>
+        <noise>
+          <type>gaussian</type>
+          <mean>0.0</mean>
+          <stddev>0.007</stddev>
+        </noise>
+      </camera>
+      <plugin name="camera_controller" filename="libgazebo_ros_camera.so">
+        <alwaysOn>true</alwaysOn>
+        <updateRate>60</updateRate>
+        <cameraName>camera7</cameraName>
+        <imageTopicName>/image_raw_7</imageTopicName>
+        <cameraInfoTopicName>camera_info</cameraInfoTopicName>
+        <frameName>camera7_Link</frameName>
         <hackBaseline>0.0</hackBaseline>
         <distortionK1>0.0</distortionK1>

Commit message: 4 vehicles

File: src/site_model/urdf/site_model.urdf.xacro (robot description, xacro)
@@ -2286,5 +2286,5 @@
   </joint>
   <!-- pillar -->
-  <link
+  <!-- <link
     name="pillar_Link">
     <inertial>
@@ -2338,5 +2338,5 @@
     <axis
       xyz="0 0 0" />
-  </joint>
+  </joint> -->
   <!-- seperate line -->
   <link

Commit message: add other 3 base links

File: src/site_model/urdf/site_model.urdf.xacro (robot description, xacro)
@@ -54,4 +54,13 @@
     <material>Gazebo/Residential</material>
   </gazebo>
+  <gazebo reference="base_Link_right">
+    <material>Gazebo/Gray</material>
+  </gazebo>
+  <gazebo reference="base_Link_left">
+    <material>Gazebo/Gray</material>
+  </gazebo>
+  <gazebo reference="base_Link_front">
+    <material>Gazebo/Gray</material>
+  </gazebo>
   <gazebo reference="pillar_Link">
     <material>Gazebo/Residential</material>
@@ -183,4 +192,166 @@
     </collision>
   </link>
+  <!-- base_link_right -->
+  <link
+    name="base_Link_right">
+    <inertial>
+      <origin
+        xyz="-1.2621568269662E-06 -1.00033198610052 -0.0249971241809568"
+        rpy="0 0 0" />
+      <mass
+        value="12481.4076184202" />
+      <inertia
+        ixx="29122.6374547981"
+        ixy="-3.27954372201533E-12"
+        ixz="3.08097412311762E-13"
+        iyy="16643.0318497451"
+        iyz="2.04194051276104E-12"
+        izz="45760.4693043086" />
+    </inertial>
+    <visual>
+      <origin
+        xyz="0 0 0"
+        rpy="0 0 0" />
+      <geometry>
+        <mesh
+          filename="package://site_model/meshes/base_link.STL" />
+      </geometry>
+      <material
+        name="">
+        <color
+          rgba="0.529411764705882 0.549019607843137 0.549019607843137 1" />
+      </material>
+    </visual>
+    <collision>
+      <origin
+        xyz="0 0 0"
+        rpy="0 0 0" />
+      <geometry>
+        <mesh
+          filename="package://site_model/meshes/base_link.STL" />
+      </geometry>
+    </collision>
+  </link>
+  <joint
+    name="base_link_right"
+    type="fixed">
+    <origin
+      xyz="4 0 0"
+      rpy="0 0 0" />
+    <parent
+      link="base_link" />
+    <child
+      link="base_Link_right" />
+    <axis
+      xyz="0 0 0" />
+  </joint>
+  <!-- base_link_left -->
+  <link
+    name="base_Link_left">
+    <inertial>
+      <origin
+        xyz="-1.2621568269662E-06 -1.00033198610052 -0.0249971241809568"
+        rpy="0 0 0" />
+      <mass
+        value="12481.4076184202" />
+      <inertia
+        ixx="29122.6374547981"
+        ixy="-3.27954372201533E-12"
+        ixz="3.08097412311762E-13"
+        iyy="16643.0318497451"
+        iyz="2.04194051276104E-12"
+        izz="45760.4693043086" />
+    </inertial>
+    <visual>
+      <origin
+        xyz="0 0 0"
+        rpy="0 0 0" />
+      <geometry>
+        <mesh
+          filename="package://site_model/meshes/base_link.STL" />
+      </geometry>
+      <material
+        name="">
+        <color
+          rgba="0.529411764705882 0.549019607843137 0.549019607843137 1" />
+      </material>
+    </visual>
+    <collision>
+      <origin
+        xyz="0 0 0"
+        rpy="0 0 0" />
+      <geometry>
+        <mesh
+          filename="package://site_model/meshes/base_link.STL" />
+      </geometry>
+    </collision>
+  </link>
+  <joint
+    name="base_link_left"
+    type="fixed">
+    <origin
+      xyz="-4 0 0"
+      rpy="0 0 0" />
+    <parent
+      link="base_link" />
+    <child
+      link="base_Link_left" />
+    <axis
+      xyz="0 0 0" />
+  </joint>
+  <!-- base_link_front -->
+  <link
+    name="base_Link_front">
+    <inertial>
+      <origin
+        xyz="-1.2621568269662E-06 -1.00033198610052 -0.0249971241809568"
+        rpy="0 0 0" />
+      <mass
+        value="12481.4076184202" />
+      <inertia
+        ixx="29122.6374547981"
+        ixy="-3.27954372201533E-12"
+        ixz="3.08097412311762E-13"
+        iyy="16643.0318497451"
+        iyz="2.04194051276104E-12"
+        izz="45760.4693043086" />
+    </inertial>
+    <visual>
+      <origin
+        xyz="0 0 0"
+        rpy="0 0 0" />
+      <geometry>
+        <mesh
+          filename="package://site_model/meshes/base_link.STL" />
+      </geometry>
+      <material
+        name="">
+        <color
+          rgba="0.529411764705882 0.549019607843137 0.549019607843137 1" />
+      </material>
+    </visual>
+    <collision>
+      <origin
+        xyz="0 0 0"
+        rpy="0 0 0" />
+      <geometry>
+        <mesh
+          filename="package://site_model/meshes/base_link.STL" />
+      </geometry>
+    </collision>
+  </link>
+  <joint
+    name="base_link_front"
+    type="fixed">
+    <origin
+      xyz="0 8 0"
+      rpy="0 0 0" />
+    <parent
+      link="base_link" />
+    <child
+      link="base_Link_front" />
+    <axis
+      xyz="0 0 0" />
+  </joint>
 <!-- Lidar11 points1 -->
   <joint name="velodyne11_base_mount_joint" type="fixed">

Commit message: improve lidcamfusion eval

File: src/site_model/urdf/site_model.urdf.xacro (robot description, xacro)
@@ -356,5 +356,5 @@
 <!-- Lidar11 points1 -->
   <joint name="velodyne11_base_mount_joint" type="fixed">
-    <origin rpy="-1.570796327 -0.7853981634 0" xyz="0 -0.475 -0.2"/>
+    <origin rpy="-1.570796327 0 0" xyz="0 -0.475 -0.2"/>
     <parent link="pole1_Link"/>
     <child link="velodyne11_base_link"/>
@@ -444,5 +444,5 @@
   <!-- Lidar12 points 2-->
   <joint name="velodyne12_base_mount_joint" type="fixed">
-    <origin rpy="-1.570796327 -0.7853981634 0" xyz="0 -0.475 1.2"/>
+    <origin rpy="-1.570796327 0 0" xyz="0 -0.475 1.2"/>
     <parent link="pole1_Link"/>
     <child link="velodyne12_base_link"/>

Commit message: fix lidar bug

File: src/site_model/urdf/site_model.urdf.xacro (robot description, xacro)
@@ -356,5 +356,5 @@
 <!-- Lidar11 points1 -->
   <joint name="velodyne11_base_mount_joint" type="fixed">
-    <origin rpy="-1.570796327 0 0" xyz="0 -0.475 -0.2"/>
+    <origin rpy="-1.570796327 -0.7853981634 0" xyz="0 -0.475 -0.2"/>
     <parent link="pole1_Link"/>
     <child link="velodyne11_base_link"/>
@@ -444,5 +444,5 @@
   <!-- Lidar12 points 2-->
   <joint name="velodyne12_base_mount_joint" type="fixed">
-    <origin rpy="-1.570796327 0 0" xyz="0 -0.475 1.2"/>
+    <origin rpy="-1.570796327 -0.7853981634 0" xyz="0 -0.475 1.2"/>
     <parent link="pole1_Link"/>
     <child link="velodyne12_base_link"/>

Commit message: update lidcamfusion eval && add camera8

File: src/site_model/urdf/site_model.urdf.xacro (robot description, xacro)
@@ -438,5 +438,5 @@
         <min_range>0.9</min_range>
         <max_range>130.0</max_range>
-        <gaussianNoise>0.02</gaussianNoise>
+        <gaussianNoise>0.006</gaussianNoise>
       </plugin>
     </sensor>
@@ -526,5 +526,5 @@
         <min_range>0.9</min_range>
         <max_range>130.0</max_range>
-        <gaussianNoise>0.02</gaussianNoise>
+        <gaussianNoise>0.006</gaussianNoise>
       </plugin>
     </sensor>
@@ -1725,4 +1725,58 @@
     </sensor>
   </gazebo>
+<!-- camera8 -->
+  <link
+    name="camera8_Link">
+    <inertial>
+      <origin
+        xyz="0.000108384331294675 -0.00200274517214477 0.0112406574811803"
+        rpy="0 0 0" />
+      <mass
+        value="0.814135587689854" />
+      <inertia
+        ixx="0.000299485503699371"
+        ixy="-8.50166027613617E-08"
+        ixz="-2.30003016200203E-09"
+        iyy="0.000280071339845325"
+        iyz="2.45106701788653E-06"
+        izz="0.000373933133462947" />
+    </inertial>
+    <visual>
+      <origin
+        xyz="-0.02 0 0"
+        rpy="0 0 0" />
+      <geometry>
+        <mesh
+          filename="package://site_model/meshes/camera8_Link.STL" />
+      </geometry>
+      <material
+        name="">
+        <color
+          rgba="0.529411764705882 0.549019607843137 0.549019607843137 1" />
+      </material>
+    </visual>
+    <collision>
+      <origin
+        xyz="0 0 0"
+        rpy="0 0 0" />
+      <geometry>
+        <mesh
+          filename="package://site_model/meshes/camera8_Link.STL" />
+      </geometry>
+    </collision>
+  </link>
+  <joint
+    name="camera8"
+    type="fixed">
+    <origin
+      xyz="0.55 2.7 0.7"
+      rpy="0 0 0.3490658503988659" />
+    <parent
+      link="base_link" />
+    <child
+      link="camera8_Link" />
+    <axis
+      xyz="0 0 0" />
+  </joint>
   <!-- Lidar_2 points3 -->
   <joint name="velodyne2_base_mount_joint" type="fixed">
@@ -1809,5 +1863,5 @@
         <min_range>0.9</min_range>
         <max_range>130.0</max_range>
-        <gaussianNoise>0.02</gaussianNoise>
+        <gaussianNoise>0.006</gaussianNoise>
       </plugin>
     </sensor>
